File: Devices/LedBar/Hardware/Boards/CenterBoard/CenterBoard.sch (KiCad schematic (older format))
At the start: 0 parts

Commit message: Added RS485 schematic sheet
Changed lines of the file:
@@
 $Descr A4 11693 8268
 encoding utf-8
-Sheet 1 2
+Sheet 1 3
 Title "LedBar - CenterBoard"
 Date "2021-04-25"
@@
 NoConn ~ 4000 2100
 NoConn ~ 4000 2200
+$Sheet
+S 2500 4000 1000 500
+U 608655BB
+F0 "RS485" 50
+F1 "RS485.sch" 50
+F2 "txd" I R 3500 4200 50
+F3 "rxd" O R 3500 4100 50
+F4 "tx_en" I R 3500 4400 50
+$EndSheet
 $EndSCHEMATC

Commit message: Added Microcontroller schematic
Connections:
- wire segments 2 -> 13
- no-connect marks 2 -> 3
Changed lines of the file:
@@
 $Descr A4 11693 8268
 encoding utf-8
-Sheet 1 3
+Sheet 1 4
 Title "LedBar - CenterBoard"
 Date "2021-04-25"
@@
 F3 "sda" B R 3500 2200 50
 $EndSheet
-Wire Wire Line
-	3500 2100 4000 2100
-Wire Wire Line
-	3500 2200 4000 2200
-NoConn ~ 4000 2100
-NoConn ~ 4000 2200
 $Sheet
 S 2500 4000 1000 500
@@
 F4 "tx_en" I R 3500 4400 50
 $EndSheet
+$Sheet
+S 4500 4000 1000 1500
+U 608B1159
+F0 "Microcontroller" 50
+F1 "Microcontroller.sch" 50
+F2 "pwm2" O R 5500 5250 50
+F3 "pwm1" O R 5500 5150 50
+F4 "rxd" I L 4500 4100 50
+F5 "txd" O L 4500 4200 50
+F6 "tx_en" O L 4500 4400 50
+F7 "~pca_oe~" O R 5500 4400 50
+F8 "scl" O R 5500 4100 50
+F9 "sda" B R 5500 4200 50
+F10 "~button~" I R 5500 4750 50
+$EndSheet
+Wire Wire Line
+	3500 4100 4500 4100
+Wire Wire Line
+	3500 4200 4500 4200
+Wire Wire Line
+	3500 4400 4500 4400
+Wire Wire Line
+	3500 2100 6000 2100
+Wire Wire Line
+	6000 2100 6000 4100
+Wire Wire Line
+	6000 4100 5500 4100
+Wire Wire Line
+	3500 2200 6100 2200
+Wire Wire Line
+	6100 2200 6100 4200
+Wire Wire Line
+	6100 4200 5500 4200
+Wire Wire Line
+	5500 4400 6500 4400
+Wire Wire Line
+	5500 4750 6500 4750
+Wire Wire Line
+	5500 5150 6500 5150
+Wire Wire Line
+	5500 5250 6500 5250
+NoConn ~ 6500 4400
+NoConn ~ 6500 5150
+NoConn ~ 6500 5250
 $EndSCHEMATC

Commit message: Added PCA schematic
Connections:
- wire segments 13 -> 19
- no-connect marks 3 -> 2
Changed lines of the file:
@@
 $Descr A4 11693 8268
 encoding utf-8
-Sheet 1 4
+Sheet 1 5
 Title "LedBar - CenterBoard"
 Date "2021-04-25"
@@
 	6100 4200 5500 4200
 Wire Wire Line
-	5500 4400 6500 4400
+	5500 4400 6300 4400
 Wire Wire Line
 	5500 4750 6500 4750
@@
 Wire Wire Line
 	5500 5250 6500 5250
-NoConn ~ 6500 4400
 NoConn ~ 6500 5150
 NoConn ~ 6500 5250
+$Sheet
+S 7000 2000 1000 1000
+U 608B2A01
+F0 "Pca" 50
+F1 "Pca.sch" 50
+F2 "scl" I L 7000 2100 50
+F3 "sda" B L 7000 2200 50
+F4 "~oe~" I L 7000 2450 50
+F5 "~button~" I L 7000 2900 50
+$EndSheet
+Connection ~ 6000 2100
+Wire Wire Line
+	6000 2100 7000 2100
+Wire Wire Line
+	6100 2200 7000 2200
+Connection ~ 6100 2200
+Wire Wire Line
+	7000 2450 6300 2450
+Wire Wire Line
+	6300 2450 6300 4400
+Wire Wire Line
+	7000 2900 6500 2900
+Wire Wire Line
+	6500 2900 6500 4750
 $EndSCHEMATC

Commit message: Added 0-10V schematic
Connections:
- no-connect marks 2 -> 0
Changed lines of the file:
@@
 $Descr A4 11693 8268
 encoding utf-8
-Sheet 1 5
+Sheet 1 6
 Title "LedBar - CenterBoard"
 Date "2021-04-25"
@@
 Wire Wire Line
 	5500 4750 6500 4750
-Wire Wire Line
-	5500 5150 6500 5150
-Wire Wire Line
-	5500 5250 6500 5250
-NoConn ~ 6500 5150
-NoConn ~ 6500 5250
 $Sheet
 S 7000 2000 1000 1000
@@
 Wire Wire Line
 	6500 2900 6500 4750
+$Sheet
+S 7000 5000 1000 500
+U 608C0E66
+F0 "0-10V" 50
+F1 "0-10V.sch" 50
+F2 "pwm1" I L 7000 5150 50
+F3 "pwm2" I L 7000 5250 50
+$EndSheet
+Wire Wire Line
+	5500 5150 7000 5150
+Wire Wire Line
+	5500 5250 7000 5250
 $EndSCHEMATC
