File: Devices/LedBar/Hardware/Boards/CenterBoard/Microcontroller.sch (KiCad schematic (older format))
At the start: 28 parts, among them J401 AVR-ISP-6, SW401 reset, U401 ATmega48PV-10AU-arduino, Y401 14.7456Mhz

Commit message: Added PCA schematic
Parts:
- renumbered TP405 to TP401, TP406 to TP402, TP401 to TP403, TP402 to TP404, TP403 to TP405, TP404 to TP406
Changed lines of the file:
@@
 $Descr A4 11693 8268
 encoding utf-8
-Sheet 4 4
+Sheet 4 5
 Title ""
 Date ""
@@
 $EndComp
 $Comp
-L power:GND #PWR0101
+L power:GND #PWR0403
 U 1 1 608B3273
 P 2500 4600
-F 0 "#PWR0101" H 2500 4350 50  0001 C CNN
+F 0 "#PWR0403" H 2500 4350 50  0001 C CNN
 F 1 "GND" H 2505 4427 50  0000 C CNN
 F 2 "" H 2500 4600 50  0001 C CNN
@@
 	2500 4600 2500 4500
 $Comp
-L power:+5V #PWR0102
+L power:+5V #PWR0404
 U 1 1 608B44A4
 P 2550 1000
-F 0 "#PWR0102" H 2550 850 50  0001 C CNN
+F 0 "#PWR0404" H 2550 850 50  0001 C CNN
 F 1 "+5V" H 2565 1173 50  0000 C CNN
 F 2 "" H 2550 1000 50  0001 C CNN
@@
 $EndComp
 $Comp
-L power:GND #PWR0103
+L power:GND #PWR0407
 U 1 1 608B81E4
 P 2900 1350
-F 0 "#PWR0103" H 2900 1100 50  0001 C CNN
+F 0 "#PWR0407" H 2900 1100 50  0001 C CNN
 F 1 "GND" V 2905 1222 50  0000 R CNN
 F 2 "" H 2900 1350 50  0001 C CNN
@@
 	2500 1350 2500 1000
 $Comp
-L power:GND #PWR0104
+L power:GND #PWR0402
 U 1 1 608B8B73
 P 2200 1350
-F 0 "#PWR0104" H 2200 1100 50  0001 C CNN
+F 0 "#PWR0402" H 2200 1100 50  0001 C CNN
 F 1 "GND" V 2205 1222 50  0000 R CNN
 F 2 "" H 2200 1350 50  0001 C CNN
@@
 $EndComp
 $Comp
-L power:GND #PWR0105
+L power:GND #PWR0401
 U 1 1 608BB07A
 P 1400 1800
-F 0 "#PWR0105" H 1400 1550 50  0001 C CNN
+F 0 "#PWR0401" H 1400 1550 50  0001 C CNN
 F 1 "GND" V 1405 1672 50  0000 R CNN
 F 2 "" H 1400 1800 50  0001 C CNN
@@
 $EndComp
 $Comp
-L power:GND #PWR0107
+L power:GND #PWR0406
 U 1 1 608DE2B0
 P 2550 6450
-F 0 "#PWR0107" H 2550 6200 50  0001 C CNN
+F 0 "#PWR0406" H 2550 6200 50  0001 C CNN
 F 1 "GND" H 2555 6277 50  0000 C CNN
 F 2 "" H 2550 6450 50  0001 C CNN
@@
 $EndComp
 $Comp
-L power:+5V #PWR0108
+L power:+5V #PWR0405
 U 1 1 608DE66D
 P 2550 5550
-F 0 "#PWR0108" H 2550 5400 50  0001 C CNN
+F 0 "#PWR0405" H 2550 5400 50  0001 C CNN
 F 1 "+5V" H 2565 5723 50  0000 C CNN
 F 2 "" H 2550 5550 50  0001 C CNN
@@
 $EndComp
 $Comp
-L power:+5V #PWR0109
+L power:+5V #PWR0409
 U 1 1 608F389F
 P 7000 1500
-F 0 "#PWR0109" H 7000 1350 50  0001 C CNN
+F 0 "#PWR0409" H 7000 1350 50  0001 C CNN
 F 1 "+5V" H 7015 1673 50  0000 C CNN
 F 2 "" H 7000 1500 50  0001 C CNN
@@
 $EndComp
 $Comp
-L power:+5V #PWR0110
+L power:+5V #PWR0412
 U 1 1 608F3FBD
 P 7500 1500
-F 0 "#PWR0110" H 7500 1350 50  0001 C CNN
+F 0 "#PWR0412" H 7500 1350 50  0001 C CNN
 F 1 "+5V" H 7515 1673 50  0000 C CNN
 F 2 "" H 7500 1500 50  0001 C CNN
@@
 	7500 1500 7500 1600
 $Comp
-L Connector:TestPoint TP401
+L Connector:TestPoint TP403
 U 1 1 608F82E1
 P 7000 2200
-F 0 "TP401" H 6942 2226 50  0000 R CNN
+F 0 "TP403" H 6942 2226 50  0000 R CNN
 F 1 "scl" H 6942 2317 50  0000 R CNN
 F 2 "AmbientLight:TestPoint_Pad_D1.0mm" H 7200 2200 50  0001 C CNN
@@
 $EndComp
 $Comp
-L Connector:TestPoint TP404
+L Connector:TestPoint TP406
 U 1 1 608FA39F
 P 7500 2200
-F 0 "TP404" H 7442 2226 50  0000 R CNN
+F 0 "TP406" H 7442 2226 50  0000 R CNN
 F 1 "sda" H 7442 2317 50  0000 R CNN
 F 2 "AmbientLight:TestPoint_Pad_D1.0mm" H 7700 2200 50  0001 C CNN
@@
 	10500 4000 9900 4000
 $Comp
-L power:GND #PWR0111
+L power:GND #PWR0414
 U 1 1 6090E71B
 P 10500 5600
-F 0 "#PWR0111" H 10500 5350 50  0001 C CNN
+F 0 "#PWR0414" H 10500 5350 50  0001 C CNN
 F 1 "GND" H 10505 5427 50  0000 C CNN
 F 2 "" H 10500 5600 50  0001 C CNN
@@
 	10150 1500 10500 1500
 $Comp
-L power:GND #PWR0112
+L power:GND #PWR0413
 U 1 1 608CBDD7
 P 10500 2600
-F 0 "#PWR0112" H 10500 2350 50  0001 C CNN
+F 0 "#PWR0413" H 10500 2350 50  0001 C CNN
 F 1 "GND" H 10505 2427 50  0000 C CNN
 F 2 "" H 10500 2600 50  0001 C CNN
@@
 $EndComp
 $Comp
-L power:+5V #PWR0113
+L power:+5V #PWR0410
 U 1 1 60908C24
 P 7000 3000
-F 0 "#PWR0113" H 7000 2850 50  0001 C CNN
+F 0 "#PWR0410" H 7000 2850 50  0001 C CNN
 F 1 "+5V" H 7015 3173 50  0000 C CNN
 F 2 "" H 7000 3000 50  0001 C CNN
@@
 $EndComp
 $Comp
-L power:GND #PWR0114
+L power:GND #PWR0411
 U 1 1 609091E4
 P 7000 4000
-F 0 "#PWR0114" H 7000 3750 50  0001 C CNN
+F 0 "#PWR0411" H 7000 3750 50  0001 C CNN
 F 1 "GND" H 7005 3827 50  0000 C CNN
 F 2 "" H 7000 4000 50  0001 C CNN
@@
 ~reset~
 $Comp
-L Connector:TestPoint TP402
+L Connector:TestPoint TP404
 U 1 1 60912AED
 P 7100 3500
-F 0 "TP402" V 7048 3688 50  0000 L CNN
+F 0 "TP404" V 7048 3688 50  0000 L CNN
 F 1 "~reset~" V 7146 3688 50  0000 L CNN
 F 2 "AmbientLight:TestPoint_Pad_D1.0mm" H 7300 3500 50  0001 C CNN
@@
 ~button~
 $Comp
-L Connector:TestPoint TP403
+L Connector:TestPoint TP405
 U 1 1 6093A750
 P 7250 4900
-F 0 "TP403" H 7192 4926 50  0000 R CNN
+F 0 "TP405" H 7192 4926 50  0000 R CNN
 F 1 "~button~" H 7192 5017 50  0000 R CNN
 F 2 "AmbientLight:TestPoint_Pad_D1.0mm" H 7450 4900 50  0001 C CNN
@@
 	3100 4200 4000 4200
 $Comp
-L Connector:TestPoint TP405
+L Connector:TestPoint TP401
 U 1 1 609CDE03
 P 4350 2800
-F 0 "TP405" V 4304 2988 50  0000 L CNN
+F 0 "TP401" V 4304 2988 50  0000 L CNN
 F 1 "dbg1" V 4395 2988 50  0000 L CNN
 F 2 "AmbientLight:TestPoint_Pad_D1.0mm" H 4550 2800 50  0001 C CNN
@@
 $EndComp
 $Comp
-L Connector:TestPoint TP406
+L Connector:TestPoint TP402
 U 1 1 609D0394
 P 4350 3100
-F 0 "TP406" V 4304 3288 50  0000 L CNN
+F 0 "TP402" V 4304 3288 50  0000 L CNN
 F 1 "dbg2" V 4395 3288 50  0000 L CNN
 F 2 "AmbientLight:TestPoint_Pad_D1.0mm" H 4550 3100 50  0001 C CNN
@@
 Connection ~ 5300 2450
 $Comp
-L power:GND #PWR0106
+L power:GND #PWR0408
 U 1 1 608D6E10
 P 5300 2450
-F 0 "#PWR0106" H 5300 2200 50  0001 C CNN
+F 0 "#PWR0408" H 5300 2200 50  0001 C CNN
 F 1 "GND" V 5305 2322 50  0000 R CNN
 F 2 "" H 5300 2450 50  0001 C CNN
