File: Devices/LedBar/Hardware/Boards/CenterBoard/Pca.sch (KiCad schematic (older format))
At the start: 26 parts, among them J501 Left, J502 Center, J503 Right, Q501 Si2302DS, Q502 Si2302DS, Q503 Si2302DS, Q504 Si2302DS, Q505 Si2302DS, Q506 Si2302DS, Q507 Si2302DS, Q508 Si2302DS, Q509 Si2302DS, Q510 Si2302DS, Q511 Si2302DS, Q512 Si2302DS, Q513 Si2302DS, Q514 Si2302DS, Q515 Si2302DS, Q516 Si2302DS, U501 PCA9685PW

Commit message: Added 0-10V schematic
Connections:
- net labels added: +12V
- wire segments 136 -> 138
Changed lines of the file:
@@
 $Descr A4 11693 8268
 encoding utf-8
-Sheet 5 5
+Sheet 5 6
 Title ""
 Date ""
@@
 Text Label 10450 3800 2    50   ~ 0
 strip4_w_out
+$Comp
+L power:+12V #PWR0101
+U 1 1 608DA5AE
+P 4000 5050
+F 0 "#PWR0101" H 4000 4900 50  0001 C CNN
+F 1 "+12V" H 4015 5223 50  0000 C CNN
+F 2 "" H 4000 5050 50  0001 C CNN
+F 3 "" H 4000 5050 50  0001 C CNN
+	1    4000 5050
+	1    0    0    -1
+$EndComp
+Wire Wire Line
+	4000 5050 4000 5150
+$Comp
+L power:+12V #PWR0102
+U 1 1 608DF9C9
+P 7500 5050
+F 0 "#PWR0102" H 7500 4900 50  0001 C CNN
+F 1 "+12V" H 7515 5223 50  0000 C CNN
+F 2 "" H 7500 5050 50  0001 C CNN
+F 3 "" H 7500 5050 50  0001 C CNN
+	1    7500 5050
+	1    0    0    -1
+$EndComp
+Wire Wire Line
+	7500 5050 7500 5150
 $EndSCHEMATC
