File: Devices/LedBar/Hardware/Boards/CenterBoard/Power.sch (KiCad schematic (older format))
At the start: 21 parts, among them J201 12V input, U201 INA219AxD, U202 AMS1117-5.0

Commit message: Added connector 15EDG-3.81-2P
Parts:
- C201, C202, C203, C205, C206, C207: footprint (none) -> Capacitor_SMD:C_0805_2012Metric_Pad1.18x1.45mm_HandSolder
- C204: footprint (none) -> Capacitor_Tantalum_SMD:CP_EIA-6032-28_Kemet-C_Pad2.25x2.35mm_HandSolder
- C208: footprint (none) -> Capacitor_Tantalum_SMD:CP_EIA-3216-18_Kemet-A_Pad1.58x1.35mm_HandSolder
- D201: footprint (none) -> Diode_SMD:D_SMB_Handsoldering
- D202: footprint (none) -> LED_SMD:LED_0805_2012Metric_Pad1.15x1.40mm_HandSolder
- R201, R203, R205: footprint (none) -> Resistor_SMD:R_0805_2012Metric_Pad1.20x1.40mm_HandSolder
- R202: footprint (none) -> Resistor_SMD:R_2512_6332Metric_Pad1.40x3.35mm_HandSolder
- R204: footprint (none) -> Resistor_SMD:R_1812_4532Metric_Pad1.30x3.40mm_HandSolder
- TP201, TP202: footprint (none) -> TestPoint:TestPoint_Pad_D1.0mm
Changed lines of the file:
@@
 F 0 "D201" V 2954 4830 50  0000 L CNN
 F 1 "SMBJ15A" V 3045 4830 50  0000 L CNN
-F 2 "" H 3000 4750 50  0001 C CNN
+F 2 "Diode_SMD:D_SMB_Handsoldering" H 3000 4750 50  0001 C CNN
 F 3 "~" H 3000 4750 50  0001 C CNN
 	1    3000 4750
@@
 F 0 "C201" H 4115 4796 50  0000 L CNN
 F 1 "0.1uF" H 4115 4705 50  0000 L CNN
-F 2 "" H 4038 4600 50  0001 C CNN
+F 2 "Capacitor_SMD:C_0805_2012Metric_Pad1.18x1.45mm_HandSolder" H 4038 4600 50  0001 C CNN
 F 3 "~" H 4000 4750 50  0001 C CNN
 	1    4000 4750
@@
 F 0 "C203" H 5115 4796 50  0000 L CNN
 F 1 "0.1uF" H 5115 4705 50  0000 L CNN
-F 2 "" H 5038 4600 50  0001 C CNN
+F 2 "Capacitor_SMD:C_0805_2012Metric_Pad1.18x1.45mm_HandSolder" H 5038 4600 50  0001 C CNN
 F 3 "~" H 5000 4750 50  0001 C CNN
 	1    5000 4750
@@
 F 0 "R202" V 4400 4000 50  0000 C CNN
 F 1 "R001/2W" V 4600 4000 50  0000 C CNN
-F 2 "" V 4430 4000 50  0001 C CNN
+F 2 "Resistor_SMD:R_2512_6332Metric_Pad1.40x3.35mm_HandSolder" V 4430 4000 50  0001 C CNN
 F 3 "~" H 4500 4000 50  0001 C CNN
 	1    4500 4000
@@
 F 0 "TP201" V 5954 4188 50  0000 L CNN
 F 1 "+12V" V 6045 4188 50  0000 L CNN
-F 2 "" H 6200 4000 50  0001 C CNN
+F 2 "TestPoint:TestPoint_Pad_D1.0mm" H 6200 4000 50  0001 C CNN
 F 3 "~" H 6200 4000 50  0001 C CNN
 	1    6000 4000
@@
 F 0 "TP202" V 9954 4688 50  0000 L CNN
 F 1 "+5V" V 10045 4688 50  0000 L CNN
-F 2 "" H 10200 4500 50  0001 C CNN
+F 2 "TestPoint:TestPoint_Pad_D1.0mm" H 10200 4500 50  0001 C CNN
 F 3 "~" H 10200 4500 50  0001 C CNN
 	1    10000 4500
@@
 F 0 "C206" H 6886 4704 50  0000 R CNN
 F 1 "0.1uF" H 6886 4795 50  0000 R CNN
-F 2 "" H 7038 4600 50  0001 C CNN
+F 2 "Capacitor_SMD:C_0805_2012Metric_Pad1.18x1.45mm_HandSolder" H 7038 4600 50  0001 C CNN
 F 3 "~" H 7000 4750 50  0001 C CNN
 	1    7000 4750
@@
 F 0 "C207" H 8115 4796 50  0000 L CNN
 F 1 "0.1uF" H 8115 4705 50  0000 L CNN
-F 2 "" H 8038 4600 50  0001 C CNN
+F 2 "Capacitor_SMD:C_0805_2012Metric_Pad1.18x1.45mm_HandSolder" H 8038 4600 50  0001 C CNN
 F 3 "~" H 8000 4750 50  0001 C CNN
 	1    8000 4750
@@
 F 0 "D202" V 10039 5132 50  0000 R CNN
 F 1 "Blue" V 9948 5132 50  0000 R CNN
-F 2 "" H 10000 5250 50  0001 C CNN
+F 2 "LED_SMD:LED_0805_2012Metric_Pad1.15x1.40mm_HandSolder" H 10000 5250 50  0001 C CNN
 F 3 "~" H 10000 5250 50  0001 C CNN
 	1    10000 5250
@@
 F 0 "R205" H 9930 4704 50  0000 R CNN
 F 1 "10k" H 9930 4795 50  0000 R CNN
-F 2 "" V 9930 4750 50  0001 C CNN
+F 2 "Resistor_SMD:R_0805_2012Metric_Pad1.20x1.40mm_HandSolder" V 9930 4750 50  0001 C CNN
 F 3 "~" H 10000 4750 50  0001 C CNN
 	1    10000 4750
@@
 F 0 "C208" H 9118 5046 50  0000 L CNN
 F 1 "10uF/10V" H 9118 4955 50  0000 L CNN
-F 2 "" H 9038 4850 50  0001 C CNN
+F 2 "Capacitor_Tantalum_SMD:CP_EIA-3216-18_Kemet-A_Pad1.58x1.35mm_HandSolder" H 9038 4850 50  0001 C CNN
 F 3 "~" H 9000 5000 50  0001 C CNN
 	1    9000 5000
@@
 F 0 "C204" H 6118 5046 50  0000 L CNN
 F 1 "10uF/16V" H 6118 4955 50  0000 L CNN
-F 2 "" H 6038 4850 50  0001 C CNN
+F 2 "Capacitor_Tantalum_SMD:CP_EIA-6032-28_Kemet-C_Pad2.25x2.35mm_HandSolder" H 6038 4850 50  0001 C CNN
 F 3 "~" H 6000 5000 50  0001 C CNN
 	1    6000 5000
@@
 F 0 "R204" H 5930 4204 50  0000 R CNN
 F 1 "100R/1W" H 5930 4295 50  0000 R CNN
-F 2 "" V 5930 4250 50  0001 C CNN
+F 2 "Resistor_SMD:R_1812_4532Metric_Pad1.30x3.40mm_HandSolder" V 5930 4250 50  0001 C CNN
 F 3 "~" H 6000 4250 50  0001 C CNN
 	1    6000 4250
@@
 F 0 "C205" H 5136 1704 50  0000 R CNN
 F 1 "0.1uF" H 5136 1795 50  0000 R CNN
-F 2 "" H 5288 1600 50  0001 C CNN
+F 2 "Capacitor_SMD:C_0805_2012Metric_Pad1.18x1.45mm_HandSolder" H 5288 1600 50  0001 C CNN
 F 3 "~" H 5250 1750 50  0001 C CNN
 	1    5250 1750
@@
 F 0 "C202" V 4248 3000 50  0000 C CNN
 F 1 "1uF" V 4339 3000 50  0000 C CNN
-F 2 "" H 4538 2850 50  0001 C CNN
+F 2 "Capacitor_SMD:C_0805_2012Metric_Pad1.18x1.45mm_HandSolder" H 4538 2850 50  0001 C CNN
 F 3 "~" H 4500 3000 50  0001 C CNN
 	1    4500 3000
@@
 F 0 "R203" H 4580 3454 50  0000 R CNN
 F 1 "10R" H 4580 3545 50  0000 R CNN
-F 2 "" V 4580 3500 50  0001 C CNN
+F 2 "Resistor_SMD:R_0805_2012Metric_Pad1.20x1.40mm_HandSolder" V 4580 3500 50  0001 C CNN
 F 3 "~" H 4650 3500 50  0001 C CNN
 	1    4650 3500
@@
 F 0 "R201" H 4281 3454 50  0000 R CNN
 F 1 "10R" H 4281 3545 50  0000 R CNN
-F 2 "" V 4280 3500 50  0001 C CNN
+F 2 "Resistor_SMD:R_0805_2012Metric_Pad1.20x1.40mm_HandSolder" V 4280 3500 50  0001 C CNN
 F 3 "~" H 4350 3500 50  0001 C CNN
 	1    4350 3500

Commit message: Added RS485 schematic sheet
Parts:
- F201: footprint (none) -> AmbientLight:Fuseholder_Cylinder-5x20mm_BLX_A_Horizontal
- J201: value 12V input -> 15EDGK-3.5/2p; footprint (none) -> AmbientLight:15EDG-3.81-2P
- TP202: footprint TestPoint:TestPoint_Pad_D1.0mm -> Package_TO_SOT_SMD:SOT-23_Handsoldering
Changed lines of the file:
@@
 $Descr A4 11693 8268
 encoding utf-8
-Sheet 2 2
+Sheet 2 3
 Title "LedBar - CenterBoard"
 Date "2021-04-25"
@@
 F 0 "F201" V 2553 4000 50  0000 C CNN
 F 1 "Max. 5A F" V 2644 4000 50  0000 C CNN
-F 2 "" V 2680 4000 50  0001 C CNN
+F 2 "AmbientLight:Fuseholder_Cylinder-5x20mm_BLX_A_Horizontal" V 2680 4000 50  0001 C CNN
 F 3 "~" H 2750 4000 50  0001 C CNN
 	1    2750 4000
@@
 P 2300 4750
 F 0 "J201" H 2408 4931 50  0000 C CNN
-F 1 "12V input" H 2250 4700 50  0000 R CNN
-F 2 "" H 2300 4750 50  0001 C CNN
-F 3 "~" H 2300 4750 50  0001 C CNN
+F 1 "15EDGK-3.5/2p" H 2250 4700 50  0000 R CNN
+F 2 "AmbientLight:15EDG-3.81-2P" H 2300 4750 50  0001 C CNN
+F 3 "https://www.on-shore.com/wp-content/uploads/OSTOQXX3251.pdf" H 2300 4750 50  0001 C CNN
 	1    2300 4750
 	1    0    0    -1
@@
 F 0 "TP202" V 9954 4688 50  0000 L CNN
 F 1 "+5V" V 10045 4688 50  0000 L CNN
-F 2 "TestPoint:TestPoint_Pad_D1.0mm" H 10200 4500 50  0001 C CNN
+F 2 "Package_TO_SOT_SMD:SOT-23_Handsoldering" H 10200 4500 50  0001 C CNN
 F 3 "~" H 10200 4500 50  0001 C CNN
 	1    10000 4500

Commit message: Added connector footprints
Parts:
- J201: value 15EDGK-3.5/2p -> 12VDC/5A; footprint AmbientLight:15EDG-3.81-2P -> AmbientLight:2EDGRC-5.08-2P
- TP202: footprint Package_TO_SOT_SMD:SOT-23_Handsoldering -> TestPoint:TestPoint_Pad_D1.0mm
Changed lines of the file:
@@
 P 2300 4750
 F 0 "J201" H 2408 4931 50  0000 C CNN
-F 1 "15EDGK-3.5/2p" H 2250 4700 50  0000 R CNN
-F 2 "AmbientLight:15EDG-3.81-2P" H 2300 4750 50  0001 C CNN
+F 1 "12VDC/5A" H 2250 4700 50  0000 R CNN
+F 2 "AmbientLight:2EDGRC-5.08-2P" H 2300 4750 50  0001 C CNN
 F 3 "https://www.on-shore.com/wp-content/uploads/OSTOQXX3251.pdf" H 2300 4750 50  0001 C CNN
 	1    2300 4750
@@
 F 0 "TP202" V 9954 4688 50  0000 L CNN
 F 1 "+5V" V 10045 4688 50  0000 L CNN
-F 2 "Package_TO_SOT_SMD:SOT-23_Handsoldering" H 10200 4500 50  0001 C CNN
+F 2 "TestPoint:TestPoint_Pad_D1.0mm" H 10200 4500 50  0001 C CNN
 F 3 "~" H 10200 4500 50  0001 C CNN
 	1    10000 4500

Commit message: Added different footprints for connectors
Parts:
- J201: footprint AmbientLight:2EDGRC-5.08-2P -> AmbientLight:15EDGRC-3.81-2P
- TP201, TP202: footprint TestPoint:TestPoint_Pad_D1.0mm -> AmbientLight:TestPoint_Pad_D1.0mm
Changed lines of the file:
@@
 F 0 "J201" H 2408 4931 50  0000 C CNN
 F 1 "12VDC/5A" H 2250 4700 50  0000 R CNN
-F 2 "AmbientLight:2EDGRC-5.08-2P" H 2300 4750 50  0001 C CNN
+F 2 "AmbientLight:15EDGRC-3.81-2P" H 2300 4750 50  0001 C CNN
 F 3 "https://www.on-shore.com/wp-content/uploads/OSTOQXX3251.pdf" H 2300 4750 50  0001 C CNN
 	1    2300 4750
@@
 F 0 "TP201" V 5954 4188 50  0000 L CNN
 F 1 "+12V" V 6045 4188 50  0000 L CNN
-F 2 "TestPoint:TestPoint_Pad_D1.0mm" H 6200 4000 50  0001 C CNN
+F 2 "AmbientLight:TestPoint_Pad_D1.0mm" H 6200 4000 50  0001 C CNN
 F 3 "~" H 6200 4000 50  0001 C CNN
 	1    6000 4000
@@
 F 0 "TP202" V 9954 4688 50  0000 L CNN
 F 1 "+5V" V 10045 4688 50  0000 L CNN
-F 2 "TestPoint:TestPoint_Pad_D1.0mm" H 10200 4500 50  0001 C CNN
+F 2 "AmbientLight:TestPoint_Pad_D1.0mm" H 10200 4500 50  0001 C CNN
 F 3 "~" H 10200 4500 50  0001 C CNN
 	1    10000 4500

Commit message: Added PCA schematic
Parts:
- added NT201: Net-Tie_2, NetTie:NetTie-2_SMD_Pad0.5mm, symbol Device:Net-Tie_2
- added TP201: gnd, AmbientLight:TestPoint_Pad_D1.0mm, symbol Connector:TestPoint
- renumbered C205 to C204, C204 to C205, TP201 to TP202, TP202 to TP203
Connections:
- net GND: now also NT201.2; no longer C201.2, C203.2, D201.2 (A), J201.2 (Pin_2)
- new net GNDPWR: C201.2, C203.2, D201.2 (A), J201.2 (Pin_2), NT201.1, TP201.1
Changed lines of the file:
@@
 $Descr A4 11693 8268
 encoding utf-8
-Sheet 2 4
+Sheet 2 5
 Title "LedBar - CenterBoard"
 Date "2021-04-25"
@@
 $EndComp
 $Comp
-L Connector:TestPoint TP201
+L Connector:TestPoint TP202
 U 1 1 608ACB83
 P 6000 4000
-F 0 "TP201" V 5954 4188 50  0000 L CNN
+F 0 "TP202" V 5954 4188 50  0000 L CNN
 F 1 "+12V" V 6045 4188 50  0000 L CNN
 F 2 "AmbientLight:TestPoint_Pad_D1.0mm" H 6200 4000 50  0001 C CNN
@@
 $EndComp
 $Comp
-L Connector:TestPoint TP202
+L Connector:TestPoint TP203
 U 1 1 608AC65D
 P 10000 4500
-F 0 "TP202" V 9954 4688 50  0000 L CNN
+F 0 "TP203" V 9954 4688 50  0000 L CNN
 F 1 "+5V" V 10045 4688 50  0000 L CNN
 F 2 "AmbientLight:TestPoint_Pad_D1.0mm" H 10200 4500 50  0001 C CNN
@@
 $EndComp
 $Comp
-L power:PWR_FLAG #FLG0203
+L power:PWR_FLAG #FLG0204
 U 1 1 608A9885
 P 7000 4500
-F 0 "#FLG0203" H 7000 4575 50  0001 C CNN
+F 0 "#FLG0204" H 7000 4575 50  0001 C CNN
 F 1 "PWR_FLAG" H 7000 4673 50  0001 C CNN
 F 2 "" H 7000 4500 50  0001 C CNN
@@
 Connection ~ 6000 4000
 $Comp
-L power:+12V #PWR0203
+L power:+12V #PWR0204
 U 1 1 608A902A
 P 6000 4000
-F 0 "#PWR0203" H 6000 3850 50  0001 C CNN
+F 0 "#PWR0204" H 6000 3850 50  0001 C CNN
 F 1 "+12V" H 6015 4173 50  0000 C CNN
 F 2 "" H 6000 4000 50  0001 C CNN
@@
 Connection ~ 10000 4500
 $Comp
-L power:+5V #PWR0205
+L power:+5V #PWR0206
 U 1 1 608A8467
 P 10000 4500
-F 0 "#PWR0205" H 10000 4350 50  0001 C CNN
+F 0 "#PWR0206" H 10000 4350 50  0001 C CNN
 F 1 "+5V" H 10015 4673 50  0000 C CNN
 F 2 "" H 10000 4500 50  0001 C CNN
@@
 $EndComp
 $Comp
-L power:GND #PWR0204
+L power:GND #PWR0205
 U 1 1 608A79AA
-P 6000 5500
-F 0 "#PWR0204" H 6000 5250 50  0001 C CNN
-F 1 "GND" H 6005 5327 50  0000 C CNN
-F 2 "" H 6000 5500 50  0001 C CNN
-F 3 "" H 6000 5500 50  0001 C CNN
-	1    6000 5500
-	1    0    0    -1
-$EndComp
-Connection ~ 6000 5500
+P 7500 5500
+F 0 "#PWR0205" H 7500 5250 50  0001 C CNN
+F 1 "GND" H 7505 5327 50  0000 C CNN
+F 2 "" H 7500 5500 50  0001 C CNN
+F 3 "" H 7500 5500 50  0001 C CNN
+	1    7500 5500
+	1    0    0    -1
+$EndComp
 Wire Wire Line
 	7000 4500 7000 4600
@@
 $EndComp
 $Comp
-L Device:CP C204
+L Device:CP C205
 U 1 1 60867727
 P 6000 5000
-F 0 "C204" H 6118 5046 50  0000 L CNN
+F 0 "C205" H 6118 5046 50  0000 L CNN
 F 1 "10uF/16V" H 6118 4955 50  0000 L CNN
 F 2 "Capacitor_Tantalum_SMD:CP_EIA-6032-28_Kemet-C_Pad2.25x2.35mm_HandSolder" H 6038 4850 50  0001 C CNN
@@
 Connection ~ 4350 4000
 $Comp
-L power:+5V #PWR0201
+L power:+5V #PWR0202
 U 1 1 608AA90C
 P 6000 1500
-F 0 "#PWR0201" H 6000 1350 50  0001 C CNN
+F 0 "#PWR0202" H 6000 1350 50  0001 C CNN
 F 1 "+5V" H 6015 1673 50  0000 C CNN
 F 2 "" H 6000 1500 50  0001 C CNN
@@
 $EndComp
 $Comp
-L power:GND #PWR0202
+L power:GND #PWR0203
 U 1 1 608AA13D
 P 6000 3000
-F 0 "#PWR0202" H 6000 2750 50  0001 C CNN
+F 0 "#PWR0203" H 6000 2750 50  0001 C CNN
 F 1 "GND" H 6005 2827 50  0000 C CNN
 F 2 "" H 6000 3000 50  0001 C CNN
@@
 sda
 $Comp
-L Device:C C205
+L Device:C C204
 U 1 1 6089F40C
 P 5250 1750
-F 0 "C205" H 5136 1704 50  0000 R CNN
+F 0 "C204" H 5136 1704 50  0000 R CNN
 F 1 "0.1uF" H 5136 1795 50  0000 R CNN
 F 2 "Capacitor_SMD:C_0805_2012Metric_Pad1.18x1.45mm_HandSolder" H 5288 1600 50  0001 C CNN
@@
 	6000 4500 6000 4850
 Wire Wire Line
-	6000 5500 7500 5500
-Wire Wire Line
 	9000 4500 10000 4500
 Connection ~ 9000 4500
@@
 	5000 4000 6000 4000
 Wire Wire Line
-	5000 5500 6000 5500
-Wire Wire Line
 	8000 4500 9000 4500
 Connection ~ 8000 4500
 Wire Wire Line
 	7500 5500 9000 5500
-Connection ~ 7500 5500
 Wire Wire Line
 	6000 2650 6000 3000
@@
 Wire Wire Line
 	4650 2350 5600 2350
+$Comp
+L power:GNDPWR #PWR?
+U 1 1 608CD0C7
+P 3000 5500
+AR Path="/608B2A01/608CD0C7" Ref="#PWR?"  Part="1"
+AR Path="/60858D7F/608CD0C7" Ref="#PWR0201"  Part="1"
+F 0 "#PWR0201" H 3000 5300 50  0001 C CNN
+F 1 "GNDPWR" H 3004 5346 50  0000 C CNN
+F 2 "" H 3000 5450 50  0001 C CNN
+F 3 "" H 3000 5450 50  0001 C CNN
+	1    3000 5500
+	1    0    0    -1
+$EndComp
+$Comp
+L Device:Net-Tie_2 NT?
+U 1 1 608CD0CD
+P 5500 5500
+AR Path="/608B2A01/608CD0CD" Ref="NT?"  Part="1"
+AR Path="/60858D7F/608CD0CD" Ref="NT201"  Part="1"
+F 0 "NT201" H 5500 5589 50  0000 C CNN
+F 1 "Net-Tie_2" H 5500 5590 50  0001 C CNN
+F 2 "NetTie:NetTie-2_SMD_Pad0.5mm" H 5500 5500 50  0001 C CNN
+F 3 "~" H 5500 5500 50  0001 C CNN
+	1    5500 5500
+	1    0    0    -1
+$EndComp
+Wire Wire Line
+	5000 5500 5400 5500
+Wire Wire Line
+	5600 5500 6000 5500
+Connection ~ 6000 5500
+Wire Wire Line
+	6000 5500 7500 5500
+Connection ~ 7500 5500
+Connection ~ 2500 5500
+$Comp
+L power:PWR_FLAG #FLG0203
+U 1 1 608D884D
+P 6000 5500
+F 0 "#FLG0203" H 6000 5575 50  0001 C CNN
+F 1 "PWR_FLAG" H 6000 5673 50  0001 C CNN
+F 2 "" H 6000 5500 50  0001 C CNN
+F 3 "~" H 6000 5500 50  0001 C CNN
+	1    6000 5500
+	-1   0    0    1
+$EndComp
+$Comp
+L Connector:TestPoint TP201
+U 1 1 608D9E42
+P 4000 5600
+F 0 "TP201" H 3942 5626 50  0000 R CNN
+F 1 "gnd" H 3942 5717 50  0000 R CNN
+F 2 "AmbientLight:TestPoint_Pad_D1.0mm" H 4200 5600 50  0001 C CNN
+F 3 "~" H 4200 5600 50  0001 C CNN
+	1    4000 5600
+	-1   0    0    1
+$EndComp
+Wire Wire Line
+	4000 5500 4000 5600
 $EndSCHEMATC
