File: Devices/LedBar/Hardware/Boards/CenterBoard/RS485.sch (KiCad schematic (older format))
At the start: 13 parts, among them J301 Conn_01x03, U301 ISO3082DW, U302 B0505S-1W-SIP4

Commit message: Added connector footprints
Parts:
- J301: value Conn_01x03 -> 15EDGK/15EDGRC; footprint (none) -> AmbientLight:15EDGRC-3.81-3P
- TP301, TP302, TP303: footprint Package_TO_SOT_SMD:SOT-23_Handsoldering -> TestPoint:TestPoint_Pad_D1.0mm
Changed lines of the file:
@@
 F 0 "TP301" H 6308 4468 50  0000 L CNN
 F 1 "txd" H 6308 4377 50  0000 L CNN
-F 2 "Package_TO_SOT_SMD:SOT-23_Handsoldering" H 6450 4350 50  0001 C CNN
+F 2 "TestPoint:TestPoint_Pad_D1.0mm" H 6450 4350 50  0001 C CNN
 F 3 "~" H 6450 4350 50  0001 C CNN
 	1    6250 4350
@@
 F 0 "TP302" H 6192 4676 50  0000 R CNN
 F 1 "rxd" H 6192 4767 50  0000 R CNN
-F 2 "Package_TO_SOT_SMD:SOT-23_Handsoldering" H 6450 4650 50  0001 C CNN
+F 2 "TestPoint:TestPoint_Pad_D1.0mm" H 6450 4650 50  0001 C CNN
 F 3 "~" H 6450 4650 50  0001 C CNN
 	1    6250 4650
@@
 F 0 "TP303" H 6192 5076 50  0000 R CNN
 F 1 "tx_en" H 6192 5167 50  0000 R CNN
-F 2 "Package_TO_SOT_SMD:SOT-23_Handsoldering" H 6450 5050 50  0001 C CNN
+F 2 "TestPoint:TestPoint_Pad_D1.0mm" H 6450 5050 50  0001 C CNN
 F 3 "~" H 6450 5050 50  0001 C CNN
 	1    6250 5050
@@
 U 1 1 60886AC6
 P 1950 4600
-F 0 "J301" H 1868 4275 50  0000 C CNN
-F 1 "Conn_01x03" H 1868 4366 50  0000 C CNN
-F 2 "" H 1950 4600 50  0001 C CNN
+F 0 "J301" H 1950 4350 50  0000 C CNN
+F 1 "15EDGK/15EDGRC" H 2350 4600 50  0000 C CNN
+F 2 "AmbientLight:15EDGRC-3.81-3P" H 1950 4600 50  0001 C CNN
 F 3 "~" H 1950 4600 50  0001 C CNN
 	1    1950 4600

Commit message: Added footprint for B0505S-1W
Parts:
- U302: footprint (none) -> AmbientLight:B0505S-1W
Changed lines of the file:
@@
 F 0 "U302" H 5000 2765 50  0000 C CNN
 F 1 "B0505S-1W-SIP4" H 5000 2674 50  0000 C CNN
-F 2 "" H 4750 2250 50  0001 C CNN
+F 2 "AmbientLight:B0505S-1W" H 4750 2250 50  0001 C CNN
 F 3 "" H 4750 2250 50  0001 C CNN
 	1    5000 2250

Commit message: Added testpoints for RS485
Parts:
- added TP301: B, TestPoint:TestPoint_Pad_D1.0mm, symbol Connector:TestPoint
- added TP302: A, TestPoint:TestPoint_Pad_D1.0mm, symbol Connector:TestPoint
- added TP303: +5V_iso, TestPoint:TestPoint_Pad_D1.0mm, symbol Connector:TestPoint
- added TP304: GND_iso, TestPoint:TestPoint_Pad_D1.0mm, symbol Connector:TestPoint
- J301: value 15EDGK/15EDGRC -> RS485
- renumbered C304 to C301, C301 to C302, C302 to C303, C303 to C304, TP301 to TP305, TP302 to TP306, TP303 to TP307
Connections:
- net +5V_iso: now also TP303.1
- net GND_iso: now also TP304.1
- net at D301.1 (A1), J301.3 (Pin_3), R301.1: now also TP301.1
- net at D301.2 (A2), J301.2 (Pin_2), R302.1: now also TP302.1
Other:
- moved on the sheet: C301, C302, C303, C304, D301, J301, R301, R302, TP305, TP306, TP307, U301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

Commit message: Added different footprints for connectors
Parts:
- C302, C303: footprint (none) -> Capacitor_Tantalum_SMD:CP_EIA-3216-18_Kemet-A_Pad1.58x1.35mm_HandSolder
- J301: footprint AmbientLight:15EDGRC-3.81-3P -> AmbientLight:15EDGRC-3.5-3P
- TP301, TP302, TP303, TP304: footprint TestPoint:TestPoint_Pad_D1.0mm -> AmbientLight:TestPoint_Pad_D1.0mm
Changed lines of the file:
@@
 F 0 "J301" H 3150 4350 50  0000 C CNN
 F 1 "RS485" H 3450 4600 50  0000 R CNN
-F 2 "AmbientLight:15EDGRC-3.81-3P" H 3150 4600 50  0001 C CNN
+F 2 "AmbientLight:15EDGRC-3.5-3P" H 3150 4600 50  0001 C CNN
 F 3 "~" H 3150 4600 50  0001 C CNN
 	1    3150 4600
@@
 F 0 "C303" H 7215 2296 50  0000 L CNN
 F 1 "4.7uF" H 7215 2205 50  0000 L CNN
-F 2 "" H 7138 2100 50  0001 C CNN
+F 2 "Capacitor_Tantalum_SMD:CP_EIA-3216-18_Kemet-A_Pad1.58x1.35mm_HandSolder" H 7138 2100 50  0001 C CNN
 F 3 "~" H 7100 2250 50  0001 C CNN
 	1    7100 2250
@@
 F 0 "C302" H 5486 2204 50  0000 R CNN
 F 1 "10uF" H 5486 2295 50  0000 R CNN
-F 2 "" H 5638 2100 50  0001 C CNN
+F 2 "Capacitor_Tantalum_SMD:CP_EIA-3216-18_Kemet-A_Pad1.58x1.35mm_HandSolder" H 5638 2100 50  0001 C CNN
 F 3 "~" H 5600 2250 50  0001 C CNN
 	1    5600 2250
@@
 F 0 "TP303" H 5058 2118 50  0000 L CNN
 F 1 "+5V_iso" H 5058 2027 50  0000 L CNN
-F 2 "TestPoint:TestPoint_Pad_D1.0mm" H 5200 2000 50  0001 C CNN
+F 2 "AmbientLight:TestPoint_Pad_D1.0mm" H 5200 2000 50  0001 C CNN
 F 3 "~" H 5200 2000 50  0001 C CNN
 	1    5000 2000
@@
 F 0 "TP304" H 4942 2526 50  0000 R CNN
 F 1 "GND_iso" H 4942 2617 50  0000 R CNN
-F 2 "TestPoint:TestPoint_Pad_D1.0mm" H 5200 2500 50  0001 C CNN
+F 2 "AmbientLight:TestPoint_Pad_D1.0mm" H 5200 2500 50  0001 C CNN
 F 3 "~" H 5200 2500 50  0001 C CNN
 	1    5000 2500
@@
 F 0 "TP301" H 3658 4468 50  0000 L CNN
 F 1 "B" H 3658 4377 50  0000 L CNN
-F 2 "TestPoint:TestPoint_Pad_D1.0mm" H 3800 4350 50  0001 C CNN
+F 2 "AmbientLight:TestPoint_Pad_D1.0mm" H 3800 4350 50  0001 C CNN
 F 3 "~" H 3800 4350 50  0001 C CNN
 	1    3600 4350
@@
 F 0 "TP302" H 3542 4676 50  0000 R CNN
 F 1 "A" H 3542 4767 50  0000 R CNN
-F 2 "TestPoint:TestPoint_Pad_D1.0mm" H 3800 4650 50  0001 C CNN
+F 2 "AmbientLight:TestPoint_Pad_D1.0mm" H 3800 4650 50  0001 C CNN
 F 3 "~" H 3800 4650 50  0001 C CNN
 	1    3600 4650

Commit message: Added Microcontroller schematic
Parts:
- TP305, TP306, TP307: footprint TestPoint:TestPoint_Pad_D1.0mm -> AmbientLight:TestPoint_Pad_D1.0mm
Changed lines of the file:
@@
 $Descr A4 11693 8268
 encoding utf-8
-Sheet 3 3
+Sheet 3 4
 Title ""
 Date ""
@@
 F 0 "TP305" H 7658 4468 50  0000 L CNN
 F 1 "txd" H 7658 4377 50  0000 L CNN
-F 2 "TestPoint:TestPoint_Pad_D1.0mm" H 7800 4350 50  0001 C CNN
+F 2 "AmbientLight:TestPoint_Pad_D1.0mm" H 7800 4350 50  0001 C CNN
 F 3 "~" H 7800 4350 50  0001 C CNN
 	1    7600 4350
@@
 F 0 "TP306" H 7542 4676 50  0000 R CNN
 F 1 "rxd" H 7542 4767 50  0000 R CNN
-F 2 "TestPoint:TestPoint_Pad_D1.0mm" H 7800 4650 50  0001 C CNN
+F 2 "AmbientLight:TestPoint_Pad_D1.0mm" H 7800 4650 50  0001 C CNN
 F 3 "~" H 7800 4650 50  0001 C CNN
 	1    7600 4650
@@
 F 0 "TP307" H 7542 5076 50  0000 R CNN
 F 1 "tx_en" H 7542 5167 50  0000 R CNN
-F 2 "TestPoint:TestPoint_Pad_D1.0mm" H 7800 5050 50  0001 C CNN
+F 2 "AmbientLight:TestPoint_Pad_D1.0mm" H 7800 5050 50  0001 C CNN
 F 3 "~" H 7800 5050 50  0001 C CNN
 	1    7600 5050
