File: Devices/LedBar/Hardware/Boards/MainBoard/Power.sch (KiCad schematic (older format))
At the start: 23 parts, among them J201 12VDC/5A, U201 INA219AxD, U202 AMS1117-5.0

Commit message: Renamed CenterBoard to MainBoard
Changed lines of the file:
@@
 encoding utf-8
 Sheet 2 6
-Title "LedBar - CenterBoard"
+Title "LedBar - MainBoard"
 Date "2021-04-25"
 Rev "0.1"
@@
 	6000 5500 7500 5500
 Connection ~ 7500 5500
-Connection ~ 2500 5500
 $Comp
 L power:PWR_FLAG #FLG0203
