File: Devices/LedBar/Hardware/Boards/MainBoard/Power.sch (KiCad schematic (older format))
At the start: 23 parts, among them J201 12VDC/5A, U201 INA219AxD, U202 AMS1117-5.0

Commit message: Added Brown-out detection
Parts:
- removed D202: Blue, LED_SMD:LED_0805_2012Metric_Pad1.15x1.40mm_HandSolder, symbol Device:LED
- removed R204: 100R/1W, Resistor_SMD:R_1812_4532Metric_Pad1.30x3.40mm_HandSolder, symbol Device:R
- removed R205: 10k, Resistor_SMD:R_0805_2012Metric_Pad1.20x1.40mm_HandSolder, symbol Device:R
Connections:
- net +12V: now also C205.1, C206.2, U202.3 (VI)
Other:
- moved on the sheet: TP203
Changed lines of the file:
@@
 	0    1    1    0
-$EndComp
-$Comp
-L Connector:TestPoint TP203
-U 1 1 608AC65D
-P 10000 4500
-F 0 "TP203" V 9954 4688 50  0000 L CNN
-F 1 "+5V" V 10045 4688 50  0000 L CNN
-F 2 "AmbientLight:TestPoint_Pad_D1.0mm" H 10200 4500 50  0001 C CNN
-F 3 "~" H 10200 4500 50  0001 C CNN
-	1    10000 4500
-	0    1    1    0
-$EndComp
-$Comp
-L power:PWR_FLAG #FLG0204
-U 1 1 608A9885
-P 7000 4500
-F 0 "#FLG0204" H 7000 4575 50  0001 C CNN
-F 1 "PWR_FLAG" H 7000 4673 50  0001 C CNN
-F 2 "" H 7000 4500 50  0001 C CNN
-F 3 "~" H 7000 4500 50  0001 C CNN
-	1    7000 4500
-	1    0    0    -1
 $EndComp
 Connection ~ 6000 4000
@@
 	1    0    0    -1
 $EndComp
-Connection ~ 10000 4500
-$Comp
-L power:+5V #PWR0206
-U 1 1 608A8467
-P 10000 4500
-F 0 "#PWR0206" H 10000 4350 50  0001 C CNN
-F 1 "+5V" H 10015 4673 50  0000 C CNN
-F 2 "" H 10000 4500 50  0001 C CNN
-F 3 "" H 10000 4500 50  0001 C CNN
-	1    10000 4500
-	1    0    0    -1
-$EndComp
 $Comp
 L power:GND #PWR0205
@@
 Wire Wire Line
 	9000 4500 9000 4850
-Wire Wire Line
-	10000 4900 10000 5100
-Wire Wire Line
-	10000 4500 10000 4600
-Wire Wire Line
-	10000 5500 10000 5400
 Wire Wire Line
 	7500 4800 7500 5000
@@
 	1    0    0    -1
 $EndComp
-Wire Wire Line
-	6000 4000 6000 4100
-$Comp
-L Device:LED D202
-U 1 1 60870EE1
-P 10000 5250
-F 0 "D202" V 10039 5132 50  0000 R CNN
-F 1 "Blue" V 9948 5132 50  0000 R CNN
-F 2 "LED_SMD:LED_0805_2012Metric_Pad1.15x1.40mm_HandSolder" H 10000 5250 50  0001 C CNN
-F 3 "~" H 10000 5250 50  0001 C CNN
-	1    10000 5250
-	0    -1   -1   0
-$EndComp
-$Comp
-L Device:R R205
-U 1 1 608702AD
-P 10000 4750
-F 0 "R205" H 9930 4704 50  0000 R CNN
-F 1 "10k" H 9930 4795 50  0000 R CNN
-F 2 "Resistor_SMD:R_0805_2012Metric_Pad1.20x1.40mm_HandSolder" V 9930 4750 50  0001 C CNN
-F 3 "~" H 10000 4750 50  0001 C CNN
-	1    10000 4750
-	-1   0    0    1
-$EndComp
 $Comp
 L Device:CP C208
@@
 	1    6000 5000
 	1    0    0    -1
-$EndComp
-$Comp
-L Device:R R204
-U 1 1 608667BE
-P 6000 4250
-F 0 "R204" H 5930 4204 50  0000 R CNN
-F 1 "100R/1W" H 5930 4295 50  0000 R CNN
-F 2 "Resistor_SMD:R_1812_4532Metric_Pad1.30x3.40mm_HandSolder" V 5930 4250 50  0001 C CNN
-F 3 "~" H 6000 4250 50  0001 C CNN
-	1    6000 4250
-	-1   0    0    1
 $EndComp
 Connection ~ 4350 4000
@@
 Connection ~ 4000 5500
 Wire Wire Line
-	6000 4400 6000 4500
-Wire Wire Line
 	6000 4500 7000 4500
 Connection ~ 6000 4500
 Wire Wire Line
 	6000 4500 6000 4850
-Wire Wire Line
-	9000 4500 10000 4500
 Connection ~ 9000 4500
-Wire Wire Line
-	9000 5500 10000 5500
-Connection ~ 9000 5500
 Connection ~ 4650 4000
 Wire Wire Line
@@
 Wire Wire Line
 	2500 4000 2500 4750
+Wire Wire Line
+	6000 4000 6000 4500
+$Comp
+L power:+5V #PWR0206
+U 1 1 608A8467
+P 9000 4500
+F 0 "#PWR0206" H 9000 4350 50  0001 C CNN
+F 1 "+5V" H 9015 4673 50  0000 C CNN
+F 2 "" H 9000 4500 50  0001 C CNN
+F 3 "" H 9000 4500 50  0001 C CNN
+	1    9000 4500
+	1    0    0    -1
+$EndComp
+$Comp
+L Connector:TestPoint TP203
+U 1 1 608AC65D
+P 9000 4500
+F 0 "TP203" V 8954 4688 50  0000 L CNN
+F 1 "+5V" V 9045 4688 50  0000 L CNN
+F 2 "AmbientLight:TestPoint_Pad_D1.0mm" H 9200 4500 50  0001 C CNN
+F 3 "~" H 9200 4500 50  0001 C CNN
+	1    9000 4500
+	0    1    1    0
+$EndComp
 $EndSCHEMATC

Commit message: Routing...
Parts:
- NT201: footprint NetTie:NetTie-2_SMD_Pad0.5mm -> NetTie:NetTie-2_THT_Pad0.3mm
Changed lines of the file:
@@
 F 0 "NT201" H 5500 5589 50  0000 C CNN
 F 1 "Net-Tie_2" H 5500 5590 50  0001 C CNN
-F 2 "NetTie:NetTie-2_SMD_Pad0.5mm" H 5500 5500 50  0001 C CNN
+F 2 "NetTie:NetTie-2_THT_Pad0.3mm" H 5500 5500 50  0001 C CNN
 F 3 "~" H 5500 5500 50  0001 C CNN
 	1    5500 5500

Commit message: Added RGBW-wire-solder-pads, removed ground-tie, routing...
Parts:
- removed NT201: Net-Tie_2, NetTie:NetTie-2_THT_Pad0.3mm, symbol Device:Net-Tie_2
Connections:
- net GNDPWR is gone; now on net GND: C201.2, C203.2, D201.2 (A), J201.1 (Pin_1), TP201.1
Changed lines of the file:
@@
-$EndComp
-$Comp
-L power:PWR_FLAG #FLG0202
-U 1 1 608AB91D
-P 5000 5500
-F 0 "#FLG0202" H 5000 5575 50  0001 C CNN
-F 1 "PWR_FLAG" H 5000 5673 50  0001 C CNN
-F 2 "" H 5000 5500 50  0001 C CNN
-F 3 "~" H 5000 5500 50  0001 C CNN
-	1    5000 5500
-	-1   0    0    1
 $EndComp
 $Comp
@@
 Wire Wire Line
 	4650 2350 5600 2350
-$Comp
-L power:GNDPWR #PWR?
-U 1 1 608CD0C7
-P 3000 5500
-AR Path="/608B2A01/608CD0C7" Ref="#PWR?"  Part="1"
-AR Path="/60858D7F/608CD0C7" Ref="#PWR0201"  Part="1"
-F 0 "#PWR0201" H 3000 5300 50  0001 C CNN
-F 1 "GNDPWR" H 3004 5346 50  0000 C CNN
-F 2 "" H 3000 5450 50  0001 C CNN
-F 3 "" H 3000 5450 50  0001 C CNN
-	1    3000 5500
-	1    0    0    -1
-$EndComp
-$Comp
-L Device:Net-Tie_2 NT?
-U 1 1 608CD0CD
-P 5500 5500
-AR Path="/608B2A01/608CD0CD" Ref="NT?"  Part="1"
-AR Path="/60858D7F/608CD0CD" Ref="NT201"  Part="1"
-F 0 "NT201" H 5500 5589 50  0000 C CNN
-F 1 "Net-Tie_2" H 5500 5590 50  0001 C CNN
-F 2 "NetTie:NetTie-2_THT_Pad0.3mm" H 5500 5500 50  0001 C CNN
-F 3 "~" H 5500 5500 50  0001 C CNN
-	1    5500 5500
-	1    0    0    -1
-$EndComp
-Wire Wire Line
-	5000 5500 5400 5500
-Wire Wire Line
-	5600 5500 6000 5500
 Connection ~ 6000 5500
 Wire Wire Line
@@
 	-1   0    0    1
 $EndComp
+Wire Wire Line
+	4000 5500 4000 5600
+Wire Wire Line
+	5000 4000 6000 4000
+Wire Wire Line
+	2500 4000 2500 4750
+Wire Wire Line
+	6000 4000 6000 4500
+$Comp
+L power:+5V #PWR0206
+U 1 1 608A8467
+P 9000 4500
+F 0 "#PWR0206" H 9000 4350 50  0001 C CNN
+F 1 "+5V" H 9015 4673 50  0000 C CNN
+F 2 "" H 9000 4500 50  0001 C CNN
+F 3 "" H 9000 4500 50  0001 C CNN
+	1    9000 4500
+	1    0    0    -1
+$EndComp
+$Comp
+L Connector:TestPoint TP203
+U 1 1 608AC65D
+P 9000 4500
+F 0 "TP203" V 8954 4688 50  0000 L CNN
+F 1 "+5V" V 9045 4688 50  0000 L CNN
+F 2 "AmbientLight:TestPoint_Pad_D1.0mm" H 9200 4500 50  0001 C CNN
+F 3 "~" H 9200 4500 50  0001 C CNN
+	1    9000 4500
+	0    1    1    0
+$EndComp
+Wire Wire Line
+	5000 5500 6000 5500
 $Comp
 L Connector:TestPoint TP201
@@
 	-1   0    0    1
 $EndComp
-Wire Wire Line
-	4000 5500 4000 5600
-Wire Wire Line
-	5000 4000 6000 4000
-Wire Wire Line
-	2500 4000 2500 4750
-Wire Wire Line
-	6000 4000 6000 4500
-$Comp
-L power:+5V #PWR0206
-U 1 1 608A8467
-P 9000 4500
-F 0 "#PWR0206" H 9000 4350 50  0001 C CNN
-F 1 "+5V" H 9015 4673 50  0000 C CNN
-F 2 "" H 9000 4500 50  0001 C CNN
-F 3 "" H 9000 4500 50  0001 C CNN
-	1    9000 4500
-	1    0    0    -1
-$EndComp
-$Comp
-L Connector:TestPoint TP203
-U 1 1 608AC65D
-P 9000 4500
-F 0 "TP203" V 8954 4688 50  0000 L CNN
-F 1 "+5V" V 9045 4688 50  0000 L CNN
-F 2 "AmbientLight:TestPoint_Pad_D1.0mm" H 9200 4500 50  0001 C CNN
-F 3 "~" H 9200 4500 50  0001 C CNN
-	1    9000 4500
-	0    1    1    0
-$EndComp
+$Comp
+L power:GNDPWR #PWR0103
+U 1 1 60965453
+P 2500 5500
+F 0 "#PWR0103" H 2500 5300 50  0001 C CNN
+F 1 "GNDPWR" H 2504 5346 50  0000 C CNN
+F 2 "" H 2500 5450 50  0001 C CNN
+F 3 "" H 2500 5450 50  0001 C CNN
+	1    2500 5500
+	1    0    0    -1
+$EndComp
+Connection ~ 2500 5500
 $EndSCHEMATC

Commit message: Routing
Connections:
- net +5V: now also U201.2 (A0); no longer U201.1 (A1)
- net GND: now also U201.1 (A1); no longer U201.2 (A0)
Changed lines of the file:
@@
 Connection ~ 6000 1500
-Wire Wire Line
-	6400 2450 6750 2450
-Wire Wire Line
-	6750 2450 6750 3000
 Wire Wire Line
 	5250 1900 5250 3000
@@
 	5250 1600 5250 1500
 Wire Wire Line
-	6000 3000 6750 3000
+	6000 3000 6650 3000
 Wire Wire Line
 	6000 1500 6750 1500
-Wire Wire Line
-	6750 1500 6750 2350
-Wire Wire Line
-	6750 2350 6400 2350
 Wire Wire Line
 	5250 1500 6000 1500
@@
 $EndComp
 Connection ~ 2500 5500
+Wire Wire Line
+	6400 2350 6650 2350
+Wire Wire Line
+	6650 2350 6650 3000
+Wire Wire Line
+	6750 2450 6400 2450
+Wire Wire Line
+	6750 1500 6750 2450
 $EndSCHEMATC

Commit message: Routing...
Connections:
- net +5V: now also U201.1 (A1); no longer U201.2 (A0)
- net GND: now also U201.2 (A0); no longer U201.1 (A1)
Changed lines of the file:
@@
 	5250 1600 5250 1500
-Wire Wire Line
-	6000 3000 6650 3000
 Wire Wire Line
 	6000 1500 6750 1500
@@
 Connection ~ 2500 5500
 Wire Wire Line
-	6400 2350 6650 2350
+	6750 1500 6750 2350
 Wire Wire Line
-	6650 2350 6650 3000
+	6750 2350 6400 2350
 Wire Wire Line
-	6750 2450 6400 2450
+	6400 2450 6750 2450
 Wire Wire Line
-	6750 1500 6750 2450
+	6750 2450 6750 3000
+Wire Wire Line
+	6000 3000 6750 3000
 $EndSCHEMATC
