File: Devices/LedBar/Hardware/Boards/MainBoard/Power.sch (KiCad schematic (older format))
At the start: 19 parts, among them J201 12VDC/5A, U201 INA219AxD, U202 AMS1117-5.0

Commit message: Work in progress
Parts:
- added TP204: gnd, AmbientLight:TestPoint_Pad_D1.0mm, symbol Connector:TestPoint
Connections:
- net +12V: no longer C205.1, C206.2, U202.3 (VI)
- net GND: now also TP204.1
- net at C201.1, D201.1 (K), F201.1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: now also C205.1, C206.2, U202.3 (VI)
Other:
- moved on the sheet: TP201, TP202
Changed lines of the file:
@@
 	5000 4900 5000 5500
 Wire Wire Line
-	4000 4600 4000 4000
+	4000 4600 4000 4500
 Wire Wire Line
 	4000 4900 4000 5500
@@
 L Connector:TestPoint TP202
 U 1 1 608ACB83
-P 6000 4000
-F 0 "TP202" V 5954 4188 50  0000 L CNN
-F 1 "+12V" V 6045 4188 50  0000 L CNN
-F 2 "AmbientLight:TestPoint_Pad_D1.0mm" H 6200 4000 50  0001 C CNN
-F 3 "~" H 6200 4000 50  0001 C CNN
-	1    6000 4000
+P 5500 4000
+F 0 "TP202" V 5454 4188 50  0000 L CNN
+F 1 "+12V" V 5545 4188 50  0000 L CNN
+F 2 "AmbientLight:TestPoint_Pad_D1.0mm" H 5700 4000 50  0001 C CNN
+F 3 "~" H 5700 4000 50  0001 C CNN
+	1    5500 4000
 	0    1    1    0
 $EndComp
-Connection ~ 6000 4000
 $Comp
 L power:+12V #PWR0204
 U 1 1 608A902A
-P 6000 4000
-F 0 "#PWR0204" H 6000 3850 50  0001 C CNN
-F 1 "+12V" H 6015 4173 50  0000 C CNN
-F 2 "" H 6000 4000 50  0001 C CNN
-F 3 "" H 6000 4000 50  0001 C CNN
-	1    6000 4000
+P 5500 4000
+F 0 "#PWR0204" H 5500 3850 50  0001 C CNN
+F 1 "+12V" H 5515 4173 50  0000 C CNN
+F 2 "" H 5500 4000 50  0001 C CNN
+F 3 "" H 5500 4000 50  0001 C CNN
+	1    5500 4000
 	1    0    0    -1
 $EndComp
@@
 Wire Wire Line
 	6000 4500 7000 4500
-Connection ~ 6000 4500
 Wire Wire Line
 	6000 4500 6000 4850
@@
 L power:PWR_FLAG #FLG0203
 U 1 1 608D884D
-P 6000 5500
-F 0 "#FLG0203" H 6000 5575 50  0001 C CNN
-F 1 "PWR_FLAG" H 6000 5673 50  0001 C CNN
-F 2 "" H 6000 5500 50  0001 C CNN
-F 3 "~" H 6000 5500 50  0001 C CNN
-	1    6000 5500
+P 5000 5500
+F 0 "#FLG0203" H 5000 5575 50  0001 C CNN
+F 1 "PWR_FLAG" H 5000 5673 50  0001 C CNN
+F 2 "" H 5000 5500 50  0001 C CNN
+F 3 "~" H 5000 5500 50  0001 C CNN
+	1    5000 5500
 	-1   0    0    1
 $EndComp
 Wire Wire Line
-	4000 5500 4000 5600
-Wire Wire Line
-	5000 4000 6000 4000
-Wire Wire Line
 	2500 4000 2500 4750
-Wire Wire Line
-	6000 4000 6000 4500
 $Comp
 L power:+5V #PWR0206
@@
 L Connector:TestPoint TP201
 U 1 1 608D9E42
-P 4000 5600
-F 0 "TP201" H 3942 5626 50  0000 R CNN
-F 1 "gnd" H 3942 5717 50  0000 R CNN
-F 2 "AmbientLight:TestPoint_Pad_D1.0mm" H 4200 5600 50  0001 C CNN
-F 3 "~" H 4200 5600 50  0001 C CNN
-	1    4000 5600
+P 9000 5600
+F 0 "TP201" H 8942 5626 50  0000 R CNN
+F 1 "gnd" H 8942 5717 50  0000 R CNN
+F 2 "AmbientLight:TestPoint_Pad_D1.0mm" H 9200 5600 50  0001 C CNN
+F 3 "~" H 9200 5600 50  0001 C CNN
+	1    9000 5600
 	-1   0    0    1
 $EndComp
@@
 Wire Wire Line
 	6000 3000 6750 3000
+Wire Wire Line
+	9000 5500 9000 5600
+Connection ~ 9000 5500
+$Comp
+L Connector:TestPoint TP204
+U 1 1 60E20AC8
+P 6000 5600
+F 0 "TP204" H 5942 5626 50  0000 R CNN
+F 1 "gnd" H 5942 5717 50  0000 R CNN
+F 2 "AmbientLight:TestPoint_Pad_D1.0mm" H 6200 5600 50  0001 C CNN
+F 3 "~" H 6200 5600 50  0001 C CNN
+	1    6000 5600
+	-1   0    0    1
+$EndComp
+Wire Wire Line
+	6000 5500 6000 5600
+Wire Wire Line
+	4000 4500 6000 4500
+Connection ~ 4000 4500
+Wire Wire Line
+	4000 4500 4000 4000
+Connection ~ 6000 4500
+Wire Wire Line
+	5000 4000 5500 4000
+Connection ~ 5500 4000
+$Comp
+L power:PWR_FLAG #FLG?
+U 1 1 60EC36EA
+P 4000 4000
+F 0 "#FLG?" H 4000 4075 50  0001 C CNN
+F 1 "PWR_FLAG" H 4000 4173 50  0001 C CNN
+F 2 "" H 4000 4000 50  0001 C CNN
+F 3 "~" H 4000 4000 50  0001 C CNN
+	1    4000 4000
+	1    0    0    -1
+$EndComp
 $EndSCHEMATC
