File: Devices/LedBar/Hardware/Boards/MainBoard/MainBoard.kicad_pcb (KiCad board)
At the start: 2 copper layers, 120 x 24 mm, 115 parts, among them J201 12VDC/5A, J301 RS485, J401 AVR-ISP-6, J501 Left, J502 Center, J503 Right, J601 0-10V(1), Q501 Si2302DS, Q502 Si2302DS, Q503 Si2302DS, Q504 Si2302DS, Q505 Si2302DS, Q506 Si2302DS, Q507 Si2302DS, Q508 Si2302DS, Q509 Si2302DS, Q510 Si2302DS, Q511 Si2302DS, Q512 Si2302DS, Q513 Si2302DS, Q514 Si2302DS, Q515 Si2302DS, Q516 Si2302DS, SW401 reset, U201 INA219AxD, U202 AMS1117-5.0, U301 ISO3082DW, U302 B0505S-1W-SIP4, U401 ATmega48PV-10AU-arduino, U501 PCA9685PW, U701 LM393, Y401 14.7456Mhz

Commit message: Routing...
Parts:
- moved TP603 121.3 mm to (98.8, 67.3), turned to 180 degrees
- moved C601 119.6 mm to (101.7, 65.3), turned to 0 degrees
- moved R601 116.9 mm to (101.7, 67.3), turned to 0 degrees
- moved TP601 112.6 mm to (104.6, 67.3), turned to 0 degrees
- moved TP701 93.2 mm to (110.0, 88.1), turned to 180 degrees
- moved R602 92.3 mm to (112.9, 84.7), turned to 0 degrees
- moved D702 88.1 mm to (112.9, 88.3), turned to 0 degrees
- moved TP501 86.9 mm to (116.5, 84.6), turned to 0 degrees
- moved R706 86.8 mm to (111.9, 91.2), turned to 90 degrees
- moved R707 83.3 mm to (113.9, 91.2), turned to 90 degrees
- moved C405 41.2 mm to (102.4, 73.3), turned to 90 degrees
- moved C404 40.0 mm to (101.7, 77.6), turned to 270 degrees
- moved TP403 38.5 mm to (125.2, 76.6)
- moved TP406 37.1 mm to (126.1, 74.2)
- moved TP404 35.2 mm to (116.3, 80.6)
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Routing:
- net GND: track 606.2 -> 606.8 mm
Other:
- board text added: "Fix test point (the footprint it self is on the wrong side)"
