File: Devices/LedBar/Hardware/Boards/MainBoard/MainBoard.kicad_pcb (KiCad board)
At the start: 2 copper layers, 120 x 24 mm, 115 parts, among them J201 12VDC/5A, J301 RS485, J401 AVR-ISP-6, J501 Left, J502 Center, J503 Right, J601 0-10V(1), Q501 Si2302DS, Q502 Si2302DS, Q503 Si2302DS, Q504 Si2302DS, Q505 Si2302DS, Q506 Si2302DS, Q507 Si2302DS, Q508 Si2302DS, Q509 Si2302DS, Q510 Si2302DS, Q511 Si2302DS, Q512 Si2302DS, Q513 Si2302DS, Q514 Si2302DS, Q515 Si2302DS, Q516 Si2302DS, SW401 reset, U201 INA219AxD, U202 AMS1117-5.0, U301 ISO3082DW, U302 B0505S-1W-SIP4, U401 ATmega48PV-10AU-arduino, U501 PCA9685PW, U701 LM393, Y401 14.7456Mhz

Commit message: Routed 0-10V and brownout circuits
Parts:
- C701, R708: moved to B.Cu
- moved R708 53.3 mm to (185.6, 101.5), turned to 180 degrees
- moved R603 47.2 mm to (193.5, 103.2), turned to 90 degrees
- moved R604 46.9 mm to (195.5, 103.2), turned to 90 degrees
- moved R605 46.9 mm to (197.6, 103.2), turned to 90 degrees
- moved C702 44.4 mm to (191.5, 103.1), turned to 90 degrees
- moved C701 42.3 mm to (194.5, 102.4)
- moved U701 38.5 mm to (195.7, 109.5), turned to 90 degrees
- moved R705 28.8 mm to (189.4, 103.2), turned to 270 degrees
- moved R703 27.2 mm to (189.4, 107.0), turned to 90 degrees
- moved R704 26.0 mm to (191.5, 107.0)
- moved D701 26.0 mm to (191.6, 111.4)
- moved R701 25.7 mm to (189.4, 110.7), turned to 270 degrees
- moved R702 24.1 mm to (189.4, 114.6), turned to 270 degrees
- moved C603 17.8 mm to (195.7, 119.4), turned to 270 degrees
- moved TP605 16.5 mm to (195.7, 116.4), turned to 90 degrees
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Connections:
- net Net-(C601-Pad1) renamed /0-10V/a1
Routing:
- net GND: track 606.8 -> 546.7 mm, vias 13 -> 17
- net /0-10V/a1: track 0.00 -> 50.9 mm, vias 0 -> 1
- net /Brown-out/~Brown_out~: track 27.6 -> 66.6 mm, vias 0 -> 1
- net Net-(C603-Pad1): track 11.1 -> 25.1 mm, vias 0 -> 1
- net +12VA: track 8.38 -> 12.1 mm, vias 0 -> 1
- net Net-(R703-Pad2): track 20.0 -> 16.3 mm
- net +12V: track 66.4 -> 68.5 mm
- net Net-(R701-Pad2): track 12.4 -> 10.3 mm
- net /Pca/strip2_r_out: track 4.21 -> 6.04 mm
- net /Pca/strip3_w_out: track 6.24 -> 7.87 mm
- net /Pca/strip2_w_out: track 6.41 -> 7.87 mm
- net /Pca/strip2_b_out: track 5.75 -> 7.00 mm
- net /Pca/strip3_b_out: track 5.49 -> 6.69 mm
- net /Pca/strip1_g_out: track 5.74 -> 6.91 mm
- net /Pca/strip2_g_out: track 4.44 -> 5.59 mm
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Other:
- board size 120 x 24 mm -> 99 x 24 mm
- board text removed: "Move 2x7 connector to correct location!!!"

Commit message: Routing
Parts:
- C401, C402, C403, C404, C405, C501, R202, R401, R403, R602, R706, R707: moved to B.Cu
- D201: moved to F.Cu
- moved TP701 87.3 mm to (190.5, 121.7), turned to 0 degrees
- moved TP603 73.9 mm to (147.9, 122.6), turned to 0 degrees
- moved TP405 71.8 mm to (174.0, 118.1), turned to 180 degrees
- moved R403 60.0 mm to (149.6, 127.7), turned to 0 degrees
- moved R401 57.0 mm to (149.6, 125.7), turned to 0 degrees
- moved C601 53.9 mm to (129.7, 111.4), turned to 270 degrees
- moved D702 52.7 mm to (153.4, 122.1), turned to 180 degrees
- moved TP402 51.8 mm to (142.5, 116.4), turned to 180 degrees
- moved R601 51.2 mm to (127.8, 111.4), turned to 270 degrees
- moved R706 51.2 mm to (154.4, 119.6), turned to 270 degrees
- moved R602 51.1 mm to (150.4, 119.4), turned to 90 degrees
- moved C401 50.1 mm to (140.6, 112.1), turned to 135 degrees
- moved C403 50.0 mm to (137.8, 109.3), turned to 315 degrees
- moved TP403 49.0 mm to (142.9, 122.2), turned to 180 degrees
- moved TP406 48.9 mm to (142.1, 120.4), turned to 180 degrees
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Connections:
- J401 pad 1: /Microcontroller/led3_miso -> /Microcontroller/led4_miso
- J401 pad 3: /Microcontroller/led4_sck -> /Microcontroller/led3_sck
- R402 pad 2: Net-(R402-Pad2) -> /Microcontroller/~reset~
- RN401 pad 5: /Microcontroller/led4_sck -> /Microcontroller/led4_miso
- RN401 pad 6: /Microcontroller/led3_miso -> /Microcontroller/led3_sck
- SW401 pad 2: Net-(R402-Pad2) -> /Microcontroller/~reset~
- U401 pad 16: /Microcontroller/led3_miso -> /Microcontroller/led4_miso
- U401 pad 17: /Microcontroller/led4_sck -> /Microcontroller/led3_sck
Routing:
- net GND: track 546.7 -> 1033.4 mm, vias 17 -> 35
- net +5V: track 38.1 -> 121.5 mm, vias 0 -> 2
- net /0-10V/a1: track 50.9 -> 102.6 mm
- net /Microcontroller/scl: track 0.00 -> 47.4 mm, vias 0 -> 1
- net /Microcontroller/~button~: track 0.00 -> 45.0 mm, vias 0 -> 1
- net /Brown-out/~Brown_out~: track 66.6 -> 109.3 mm, vias 1 -> 3
- net /Microcontroller/sda: track 0.00 -> 40.2 mm, vias 0 -> 1
- net /Microcontroller/led4_miso: track 0.00 -> 38.3 mm, vias 0 -> 1
- net /Pca/~oe~: track 0.00 -> 33.3 mm, vias 0 -> 4
- net /Microcontroller/tx_en: track 3.92 -> 33.5 mm
- net /Microcontroller/txd: track 3.59 -> 31.4 mm
- net /Microcontroller/rxd: track 2.65 -> 28.0 mm
- net /Microcontroller/led3_sck: track 0.00 -> 23.9 mm
- net /Microcontroller/addr5: track 8.78 -> 31.8 mm, vias 0 -> 1
- net /Microcontroller/led2_mosi: track 0.00 -> 22.2 mm
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- added copper zone on B.Cu, net +12V
- added copper zone on B.Cu, net Net-(C201-Pad1)

Commit message: Fixed testpoint footprint
Parts:
- TP201, TP202, TP203, TP301, TP302, TP303, TP304, TP305, TP306, TP307, TP401, TP402, TP403, TP404, TP405, TP501, TP601, TP603, TP605, TP701: moved to B.Cu
- turned TP605 to 270 degrees
Connections:
- U201 pad 1: +5V -> GND
- U201 pad 2: GND -> +5V
- U301 pad 11: (no net) -> Net-(U301-Pad11)
- U301 pad 14: (no net) -> Net-(U301-Pad14)
- U401 pad 19: (no net) -> Net-(U401-Pad19)
- U401 pad 22: (no net) -> Net-(U401-Pad22)

Commit message: Routing...
Parts:
- R401, R403: moved to F.Cu
- moved C201 20.2 mm to (144.4, 106.0), turned to 180 degrees
- moved C203 16.1 mm to (144.4, 108.1), turned to 180 degrees
- moved TP202 13.3 mm to (159.6, 102.2), turned to 180 degrees
- moved TP501 4.13 mm to (145.4, 116.9)
- moved R403 4.08 mm to (145.7, 126.5), turned to 90 degrees
- moved D201 4.06 mm to (140.0, 105.3)
- moved R202 2.14 mm to (147.3, 102.6), turned to 180 degrees
- moved C202 1.02 mm to (151.1, 107.0)
- moved R201 1.02 mm to (148.2, 106.0)
- moved R203 1.02 mm to (148.2, 108.1)
- moved R401 0.57 mm to (149.5, 126.2), turned to 270 degrees
- moved C208 0.13 mm to (113.8, 105.2)
- turned C204 to 270 degrees
Connections:
- U201 pad 1: GND -> +5V
- U201 pad 2: +5V -> GND
- U301 pad 11: Net-(U301-Pad11) -> (no net)
- U301 pad 14: Net-(U301-Pad14) -> (no net)
- U401 pad 19: Net-(U401-Pad19) -> (no net)
- U401 pad 22: Net-(U401-Pad22) -> (no net)
Routing:
- net GND: track 1033.4 -> 1057.1 mm, vias 35 -> 43
- net Net-(C201-Pad1): track 7.76 -> 14.8 mm
- net +12V: track 75.5 -> 80.6 mm
- net +5V: track 121.5 -> 119.9 mm, vias 2 -> 4
- net /Pca/~oe~: track 33.3 -> 33.9 mm
- net /Microcontroller/sda: track 40.2 -> 40.9 mm

Commit message: cleaning layout
Parts:
- TP406: moved to B.Cu
- moved D201 1.47 mm to (138.5, 105.3)
- moved Q510 0.79 mm to (180.7, 116.4)
- moved F201 0.79 mm to (131.9, 105.5)
- moved R601 0.66 mm to (127.8, 112.0)
- moved Q513 0.55 mm to (186.6, 119.9)
- moved C502 0.47 mm to (182.7, 106.5)
- moved C503 0.46 mm to (182.7, 104.0)
- moved Q514 0.46 mm to (178.0, 119.9)
- moved Q509 0.41 mm to (186.6, 116.4)
- moved J502 0.34 mm to (173.3, 103.6)
- moved Q501 0.32 mm to (186.6, 112.9)
- moved Q502 0.25 mm to (180.7, 112.9)
Routing:
- net GND: track 1057.1 -> 989.6 mm, vias 43 -> 62
- net +5V: track 119.9 -> 126.2 mm, vias 4 -> 3
- net +12V: track 80.6 -> 85.5 mm
- net /Pca/strip1_b: track 32.2 -> 34.4 mm
- net /Pca/strip1_r: track 38.9 -> 40.6 mm
- net /Pca/strip1_b_out: track 8.33 -> 9.56 mm
- net /Pca/strip1_g: track 40.8 -> 42.0 mm
- net /Pca/~oe~: track 33.9 -> 32.9 mm
- net /Pca/strip2_b_out: track 7.00 -> 7.97 mm
- net /Pca/strip2_g: track 35.5 -> 36.4 mm
- net /Pca/strip2_w_out: track 7.87 -> 8.78 mm
- net /Microcontroller/led4_miso: track 38.3 -> 37.5 mm
- net Net-(C201-Pad1): track 14.8 -> 14.1 mm

Commit message: Cleaning layout
Parts:
- moved C202 1.42 mm to (152.2, 106.0)
- moved R201 1.09 mm to (149.3, 106.0)
- moved R203 1.09 mm to (149.3, 108.1)
- moved U201 1.09 mm to (156.0, 107.4)
- moved C201 1.09 mm to (145.5, 106.0)
- moved C203 1.09 mm to (145.5, 108.1)
- moved C204 1.09 mm to (159.7, 105.9)
- moved C505 0.97 mm to (165.9, 104.0)
- moved C504 0.94 mm to (165.9, 106.4)
- moved Q515 0.46 mm to (170.1, 119.9)
- moved Q503 0.44 mm to (168.4, 112.9)
- moved Q511 0.36 mm to (168.4, 116.4)
- moved R708 0.20 mm to (189.4, 102.6)
Routing:
- net GND: track 989.6 -> 965.1 mm, vias 62 -> 63
- net +12V: track 85.5 -> 76.6 mm
- net +5V: track 126.2 -> 130.3 mm, vias 3 -> 4
- net Net-(F201-Pad2): track 10.2 -> 8.61 mm
- net /Pca/strip3_r: track 11.5 -> 12.8 mm
- net /Microcontroller/scl: track 47.4 -> 48.5 mm
- net /Microcontroller/sda: track 40.9 -> 41.7 mm
- net /Pca/strip3_w_out: track 7.87 -> 7.20 mm
- net /0-10V/a1: track 102.9 -> 102.3 mm

Commit message: Routing
Parts:
- moved Q504 0.77 mm to (162.6, 112.9)
- moved Q516 0.46 mm to (158.4, 119.9)
- moved J503 0.39 mm to (155.8, 105.6)
- moved Q507 0.35 mm to (169.4, 108.5)
- moved Q512 0.28 mm to (160.3, 116.4)
- moved J501 0.24 mm to (192.9, 105.6)
- moved R201 0.08 mm to (149.3, 106.0)
- moved R203 0.08 mm to (149.3, 108.1)
- turned C204 to 90 degrees
Routing:
- net GND: track 965.1 -> 912.6 mm, vias 63 -> 64
- net +12V: track 76.6 -> 69.9 mm
- net /Pca/strip4_b_out: track 9.34 -> 7.04 mm
- net +5V: track 130.3 -> 129.0 mm
- net Net-(C603-Pad1): track 25.3 -> 26.0 mm
- net /Microcontroller/~button~: track 45.3 -> 44.7 mm
- net /Pca/strip4_w_out: track 8.34 -> 7.83 mm
- net /Pca/strip4_g_out: track 6.06 -> 6.56 mm

Commit message: Added Rtc
Parts:
- added BT801: 3V, Battery:Battery_Panasonic_CR1220-VCN_Vertical_CircularHoles, F.Cu at (141.3, 93.2)
- added U801: DS1307Z+, Package_SO:SOIC-8_3.9x4.9mm_P1.27mm, F.Cu at (146.7, 117.7)
- added Y801: 23.768kHz, Crystal:Crystal_C38-LF_D3.0mm_L8.0mm_Vertical, F.Cu at (145.5, 96.0)
- moved TP501 3.60 mm to (144.8, 120.4)
- moved R602 2.97 mm to (148.9, 122.0), turned to 180 degrees
- moved TP603 1.87 mm to (146.1, 122.1)
- moved Q508 0.51 mm to (161.3, 108.5)
- moved J503 0.36 mm to (156.1, 105.6)
Routing:
- net GND: track 912.6 -> 948.4 mm, vias 64 -> 67
- net /Microcontroller/scl: track 48.5 -> 57.3 mm
- net /Microcontroller/sda: track 41.7 -> 49.1 mm
- net +12V: track 69.9 -> 63.7 mm
- net /0-10V/a1: track 102.3 -> 107.0 mm
- net Net-(BT801-Pad1): track 0.00 -> 3.74 mm
- net /Brown-out/~Brown_out~: track 109.2 -> 106.0 mm
- net /Pca/~oe~: track 32.9 -> 35.0 mm, vias 4 -> 3
- net Net-(U801-Pad1): track 0.00 -> 2.15 mm
- net Net-(U801-Pad2): track 0.00 -> 1.89 mm
- net /Pca/strip4_r_out: track 7.00 -> 8.88 mm
- net /Pca/strip4_g: track 10.8 -> 12.0 mm
- net Net-(D702-Pad2): track 5.44 -> 4.38 mm
- net /Pca/strip4_b_out: track 7.04 -> 7.79 mm
