File: Devices/LedBar/Hardware/Boards/MainBoard/MainBoard.kicad_pcb (KiCad board)
At the start: 2 copper layers, 99 x 24 mm, 118 parts, among them J201 12VDC/5A, J301 RS485, J401 AVR-ISP-6, J501 Left, J502 Center, J503 Right, J601 0-10V(1), Q501 Si2302DS, Q502 Si2302DS, Q503 Si2302DS, Q504 Si2302DS, Q505 Si2302DS, Q506 Si2302DS, Q507 Si2302DS, Q508 Si2302DS, Q509 Si2302DS, Q510 Si2302DS, Q511 Si2302DS, Q512 Si2302DS, Q513 Si2302DS, Q514 Si2302DS, Q515 Si2302DS, Q516 Si2302DS, SW401 reset, U201 INA219AxD, U202 AMS1117-5.0, U301 ISO3082DW, U302 B0505S-1W-SIP4, U401 ATmega48PV-10AU-arduino, U501 PCA9685PW, U701 LM393, U801 DS1307Z+, Y401 14.7456Mhz, Y801 23.768kHz

Commit message: Removed RTC and EEPROM all routed
Parts:
- removed BT801: 3V, Battery:Battery_Panasonic_CR1220-VCN_Vertical_CircularHoles
- removed U801: DS1307Z+, Package_SO:SOIC-8_3.9x4.9mm_P1.27mm
- removed Y801: 23.768kHz, Crystal:Crystal_C38-LF_D3.0mm_L8.0mm_Vertical
- moved R403 9.55 mm to (146.6, 117.0), turned to 270 degrees
- moved R401 9.22 mm to (148.6, 117.0)
- moved R602 2.69 mm to (147.1, 120.1)
- moved R707 1.93 mm to (150.5, 119.6)
- moved C603 1.84 mm to (193.9, 119.4)
- moved J501 1.84 mm to (191.1, 105.6)
- moved J601 1.84 mm to (191.2, 116.6)
- moved Q502 1.84 mm to (178.9, 112.9)
- moved Q510 1.84 mm to (178.9, 116.4)
- moved R201 1.84 mm to (147.4, 106.0)
- moved R203 1.84 mm to (147.4, 108.1)
- moved R605 1.84 mm to (195.7, 103.2)
- moved TP605 1.84 mm to (193.9, 116.4)
- moved C201 1.84 mm to (143.6, 106.0)
- moved C202 1.84 mm to (150.4, 106.0)
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Routing:
- net GND: track 948.4 -> 920.8 mm, vias 67 -> 76
- net /Microcontroller/scl: track 57.3 -> 47.9 mm
- net /Microcontroller/sda: track 49.1 -> 41.7 mm
- net Net-(BT801-Pad1): track 3.74 -> 0.00 mm
- net /Pca/~oe~: track 35.0 -> 31.6 mm
- net +5V: track 129.0 -> 132.1 mm
- net GND_iso: track 8.86 -> 6.55 mm
- net /Brown-out/~Brown_out~: track 106.0 -> 108.2 mm
- net Net-(U801-Pad1): track 2.15 -> 0.00 mm
- net Net-(U801-Pad2): track 1.89 -> 0.00 mm
- net +12V: track 63.7 -> 61.9 mm
- net /0-10V/a1: track 107.0 -> 108.6 mm
- net /Microcontroller/~button~: track 44.7 -> 43.2 mm
- net Net-(C201-Pad1): track 14.1 -> 14.9 mm
- net +5V_iso: track 14.0 -> 14.5 mm
Other:
- board size 99 x 24 mm -> 97.2 x 24 mm

Commit message: Work in progress
Parts:
- added TP204: gnd, AmbientLight:TestPoint_Pad_D1.0mm, B.Cu at (162.2, 110.2)
- added TP407: gnd, AmbientLight:TestPoint_Pad_D1.0mm, B.Cu at (146.6, 116.7)
- added TP408: gnd, AmbientLight:TestPoint_Pad_D1.0mm, B.Cu at (172.4, 120.8)
- added TP502: strip1_w, AmbientLight:TestPoint_Pad_D1.0mm, B.Cu at (181.0, 119.9)
- added TP503: strip1_w_out, AmbientLight:TestPoint_Pad_D1.0mm, B.Cu at (188.5, 118.9)
- added TP504: gnd, AmbientLight:TestPoint_Pad_D1.0mm, B.Cu at (188.5, 121.0)
- moved TP701 40.8 mm to (148.1, 118.1)
- moved TP603 9.99 mm to (145.7, 112.4)
- moved TP201 8.73 mm to (111.8, 108.7)
- moved TP202 4.74 mm to (162.2, 104.0)
- moved TP405 0.75 mm to (172.4, 118.8)
- moved TP402 0.32 mm to (142.2, 116.4)
- moved C403 0.07 mm to (137.9, 109.3)
- moved R605 0.07 mm to (195.7, 103.2)
Connections:
- C205 pad 1: +12V -> Net-(C201-Pad1)
- C206 pad 2: +12V -> Net-(C201-Pad1)
- R701 pad 1: +12V -> +12VA
- R703 pad 1: +12V -> +12VA
- U202 pad 3: +12V -> Net-(C201-Pad1)
Routing:
- net +12V: track 61.9 -> 24.8 mm
- net GND: track 920.8 -> 895.1 mm, vias 76 -> 84
- net Net-(C201-Pad1): track 14.9 -> 26.6 mm
- net +12VA: track 15.0 -> 25.4 mm
- net /Brown-out/~Brown_out~: track 108.2 -> 111.8 mm
- net +5V: track 132.1 -> 129.8 mm
- net /Pca/strip1_w_out: track 10.3 -> 11.8 mm
- net /Microcontroller/led2_mosi: track 22.2 -> 23.5 mm
- net Net-(C603-Pad1): track 26.0 -> 25.1 mm
- net /Microcontroller/~button~: track 43.2 -> 43.9 mm
- net /Microcontroller/addr1: track 18.7 -> 19.2 mm
- net GND_iso: vias 3 -> 4
Other:
- board text added: "LSB"
- board text added: "Reset"

Commit message: Added resistor on PCB, updated coper-plane and updated silkscreen
Parts:
- added R303: 56, Resistor_SMD:R_1206_3216Metric, B.Cu at (102.5, 111.0)
- moved TP301 1.67 mm to (103.5, 113.2)
- moved TP202 0.96 mm to (162.1, 105.0)
- moved TP302 0.85 mm to (103.5, 116.7)
- moved TP304 0.19 mm to (103.5, 120.1)
- moved TP204 0.05 mm to (162.2, 110.2)
Routing:
- net GND: track 895.1 -> 903.5 mm, vias 84 -> 85
- net +5V_iso: track 14.5 -> 19.0 mm
- net /RS485/B: track 11.4 -> 10.5 mm
- net /RS485/A: track 13.8 -> 13.3 mm
Other:
- board text added: "Created by: Roel Drost Revision: ${rev} (${rev_date}) https://github.com/Roel1983/LEDBar2"
- board text added: "LEDBar - MainBoard"
