File: Devices/LedBar/Hardware/Boards/MainBoard/Microcontroller.sch (KiCad schematic (older format))
At the start: 28 parts, among them J401 AVR-ISP-6, SW401 reset, U401 ATmega48PV-10AU-arduino, Y401 14.7456Mhz

Commit message: Fixed using wrong resistor network symbol
Parts:
- RN401: symbol Device:R_Network04_Split -> Device:R_Pack04_Split
Connections:
- net labels removed: led2, led3, led4
Other:
- moved on the sheet: RN401B, RN401C, RN401D
Changed lines of the file:
@@
 addr5
 $Comp
-L Device:R_Network04_Split RN401
+L Device:R_Pack04_Split RN401
 U 1 1 60918B02
 P 9500 1000
@@
 $EndComp
 $Comp
-L Device:R_Network04_Split RN401
+L Device:R_Pack04_Split RN401
 U 2 1 608B38B6
 P 9500 1500
@@
 $EndComp
 $Comp
-L Device:R_Network04_Split RN401
+L Device:R_Pack04_Split RN401
 U 3 1 608B3CF0
 P 9500 2000
@@
 $EndComp
 $Comp
-L Device:R_Network04_Split RN401
+L Device:R_Pack04_Split RN401
 U 4 1 608B3FC7
 P 9500 2500
@@
 	0    -1   1    0
 $EndComp
-Wire Wire Line
-	9000 1000 9350 1000
-Wire Wire Line
-	9000 1500 9350 1500
-Wire Wire Line
-	9000 2000 9350 2000
-Wire Wire Line
-	9000 2500 9350 2500
 $Comp
 L Device:LED D401
@@
 Wire Wire Line
 	10500 2000 10500 2500
-Text Label 9050 1000 0    50   ~ 0
+Text Label 8800 1000 0    50   ~ 0
 led1
-Text Label 9050 1500 0    50   ~ 0
-led2
-Text Label 9050 2000 0    50   ~ 0
-led3
-Text Label 9050 2500 0    50   ~ 0
-led4
 $Comp
 L Device:R R402
@@
 	0    -1   -1   0
 $EndComp
+Text Label 8800 1500 0    50   ~ 0
+led2_mosi
+Text Label 8800 2000 0    50   ~ 0
+led3_miso
+Text Label 8800 2500 0    50   ~ 0
+led4_sck
+Wire Wire Line
+	8750 1000 9350 1000
+Wire Wire Line
+	8750 1500 9350 1500
+Wire Wire Line
+	8750 2000 9350 2000
+Wire Wire Line
+	8750 2500 9350 2500
 $EndSCHEMATC

Commit message: Added Brown-out detection
Parts:
- added R602: 10k, Resistor_SMD:R_0805_2012Metric_Pad1.20x1.40mm_HandSolder, symbol Device:R
Connections:
- net labels added: ~brown_out~
- net labels removed: pwm2
- wire segments 91 -> 94
- no-connect marks 2 -> 3
Changed lines of the file:
@@
 $Descr A4 11693 8268
 encoding utf-8
-Sheet 4 6
+Sheet 6 6
 Title "LedBar - MainBoard"
 Date "2021-04-25"
@@
 Wire Wire Line
 	1500 1800 1400 1800
-Text HLabel 4000 4100 2    50   Output ~ 0
-pwm2
 Text HLabel 4000 4000 2    50   Output ~ 0
 pwm1
@@
 Text HLabel 4000 3000 2    50   Output ~ 0
 tx_en
-Text HLabel 4000 3700 2    50   Output ~ 0
+Text HLabel 5500 3700 2    50   Output ~ 0
 ~pca_oe~
 Text Label 3500 3800 0    50   ~ 0
@@
 	3100 3600 4000 3600
 Wire Wire Line
-	3100 3700 4000 3700
+	3100 3700 5000 3700
 Wire Wire Line
 	3100 3800 4000 3800
@@
 Wire Wire Line
 	3100 4000 4000 4000
-Wire Wire Line
-	3100 4100 4000 4100
 Wire Wire Line
 	3100 4200 4000 4200
@@
 Wire Wire Line
 	8750 2500 9350 2500
+NoConn ~ 3100 4100
+Text HLabel 5500 3900 2    50   Input ~ 0
+~brown_out~
+$Comp
+L Device:R R602
+U 1 1 60945A82
+P 5250 3900
+F 0 "R602" V 5350 3850 50  0000 L CNN
+F 1 "10k" V 5150 3900 50  0000 C CNN
+F 2 "Resistor_SMD:R_0805_2012Metric_Pad1.20x1.40mm_HandSolder" V 5180 3900 50  0001 C CNN
+F 3 "~" H 5250 3900 50  0001 C CNN
+	1    5250 3900
+	0    1    1    0
+$EndComp
+Wire Wire Line
+	5500 3900 5400 3900
+Wire Wire Line
+	5100 3900 5000 3900
+Wire Wire Line
+	5000 3900 5000 3700
+Connection ~ 5000 3700
+Wire Wire Line
+	5000 3700 5500 3700
 $EndSCHEMATC

Commit message: Moved brown-out to it own sheet
Connections:
- wire segments 94 -> 95
Other:
- moved on the sheet: R602
Changed lines of the file:
@@
 $Descr A4 11693 8268
 encoding utf-8
-Sheet 6 6
+Sheet 6 7
 Title "LedBar - MainBoard"
 Date "2021-04-25"
@@
 Text HLabel 4000 3000 2    50   Output ~ 0
 tx_en
-Text HLabel 5500 3700 2    50   Output ~ 0
+Text HLabel 7500 5500 2    50   Output ~ 0
 ~pca_oe~
 Text Label 3500 3800 0    50   ~ 0
@@
 	3100 3600 4000 3600
 Wire Wire Line
-	3100 3700 5000 3700
-Wire Wire Line
 	3100 3800 4000 3800
 Wire Wire Line
@@
 	8750 2500 9350 2500
 NoConn ~ 3100 4100
-Text HLabel 5500 3900 2    50   Input ~ 0
+Text HLabel 6500 5700 0    50   Input ~ 0
 ~brown_out~
 $Comp
 L Device:R R602
 U 1 1 60945A82
-P 5250 3900
-F 0 "R602" V 5350 3850 50  0000 L CNN
-F 1 "10k" V 5150 3900 50  0000 C CNN
-F 2 "Resistor_SMD:R_0805_2012Metric_Pad1.20x1.40mm_HandSolder" V 5180 3900 50  0001 C CNN
-F 3 "~" H 5250 3900 50  0001 C CNN
-	1    5250 3900
-	0    1    1    0
-$EndComp
-Wire Wire Line
-	5500 3900 5400 3900
-Wire Wire Line
-	5100 3900 5000 3900
-Wire Wire Line
-	5000 3900 5000 3700
-Connection ~ 5000 3700
-Wire Wire Line
-	5000 3700 5500 3700
+P 7000 5700
+F 0 "R602" V 7100 5700 50  0000 C CNN
+F 1 "10k" V 6900 5700 50  0000 C CNN
+F 2 "Resistor_SMD:R_0805_2012Metric_Pad1.20x1.40mm_HandSolder" V 6930 5700 50  0001 C CNN
+F 3 "~" H 7000 5700 50  0001 C CNN
+	1    7000 5700
+	0    1    1    0
+$EndComp
+Text Label 3500 3700 0    50   ~ 0
+~pca_oe~
+Wire Wire Line
+	3100 3700 4000 3700
+Wire Wire Line
+	6500 5700 6850 5700
+Wire Wire Line
+	7150 5700 7250 5700
+Wire Wire Line
+	7250 5700 7250 5500
+Wire Wire Line
+	7250 5500 7500 5500
+Wire Wire Line
+	6500 5500 7250 5500
+Connection ~ 7250 5500
+Text Label 6550 5500 0    50   ~ 0
+~pca_oe~
 $EndSCHEMATC

Commit message: FETs routed
Connections:
- wire segments 95 -> 97
- no-connect marks 3 -> 2
Other:
- moved on the sheet: R602
Changed lines of the file:
@@
 Text HLabel 7500 5500 2    50   Output ~ 0
 ~pca_oe~
-Text Label 3500 3800 0    50   ~ 0
+Text Label 3500 3900 0    50   ~ 0
 addr1
-Text Label 3500 3900 0    50   ~ 0
+Text Label 3500 4100 0    50   ~ 0
 addr2
 Text Label 3500 4200 0    50   ~ 0
@@
 Wire Wire Line
 	8750 2500 9350 2500
-NoConn ~ 3100 4100
-Text HLabel 6500 5700 0    50   Input ~ 0
+Text HLabel 7500 6000 2    50   Input ~ 0
 ~brown_out~
 $Comp
 L Device:R R602
 U 1 1 60945A82
-P 7000 5700
-F 0 "R602" V 7100 5700 50  0000 C CNN
-F 1 "10k" V 6900 5700 50  0000 C CNN
-F 2 "Resistor_SMD:R_0805_2012Metric_Pad1.20x1.40mm_HandSolder" V 6930 5700 50  0001 C CNN
-F 3 "~" H 7000 5700 50  0001 C CNN
-	1    7000 5700
-	0    1    1    0
+P 7250 5750
+F 0 "R602" H 7200 5700 50  0000 R CNN
+F 1 "10k" H 7200 5800 50  0000 R CNN
+F 2 "Resistor_SMD:R_0805_2012Metric_Pad1.20x1.40mm_HandSolder" V 7180 5750 50  0001 C CNN
+F 3 "~" H 7250 5750 50  0001 C CNN
+	1    7250 5750
+	-1   0    0    1
 $EndComp
 Text Label 3500 3700 0    50   ~ 0
@@
 Wire Wire Line
 	3100 3700 4000 3700
-Wire Wire Line
-	6500 5700 6850 5700
-Wire Wire Line
-	7150 5700 7250 5700
-Wire Wire Line
-	7250 5700 7250 5500
-Wire Wire Line
-	7250 5500 7500 5500
-Wire Wire Line
-	6500 5500 7250 5500
-Connection ~ 7250 5500
 Text Label 6550 5500 0    50   ~ 0
 ~pca_oe~
+Text Label 6550 6000 0    50   ~ 0
+~brown_out~
+Text Label 3500 3800 0    50   ~ 0
+~brown_out~
+Wire Wire Line
+	3100 4100 4000 4100
+Wire Wire Line
+	6500 6000 7250 6000
+Wire Wire Line
+	6500 5500 7250 5500
+Wire Wire Line
+	7250 5500 7250 5600
+Connection ~ 7250 5500
+Wire Wire Line
+	7250 5500 7500 5500
+Wire Wire Line
+	7250 5900 7250 6000
+Connection ~ 7250 6000
+Wire Wire Line
+	7250 6000 7500 6000
 $EndSCHEMATC

Commit message: Routing...
Parts:
- SW401: footprint Resistor_SMD:R_0805_2012Metric_Pad1.20x1.40mm_HandSolder -> Button_Switch_SMD:SW_SPST_CK_RS282G05A3
Changed lines of the file:
@@
 F 0 "SW401" V 7046 3702 50  0000 R CNN
 F 1 "reset" V 6955 3702 50  0000 R CNN
-F 2 "Resistor_SMD:R_0805_2012Metric_Pad1.20x1.40mm_HandSolder" H 7000 3950 50  0001 C CNN
+F 2 "Button_Switch_SMD:SW_SPST_CK_RS282G05A3" H 7000 3950 50  0001 C CNN
 F 3 "~" H 7000 3950 50  0001 C CNN
 	1    7000 3750

Commit message: Routing
Connections:
- net labels added: led3_sck, led4_miso
- net labels removed: led3_miso, led4_sck
- wire segments 97 -> 99
Changed lines of the file:
@@
 led2_mosi
 Text Label 3500 2200 0    50   ~ 0
-led3_miso
+led4_miso
 Text Label 3500 2300 0    50   ~ 0
-led4_sck
+led3_sck
 Text Label 3500 2700 0    50   ~ 0
 ~button~
@@
 	7000 3950 7000 4000
 Wire Wire Line
-	7000 3550 7000 3400
+	7000 3550 7000 3500
 Wire Wire Line
 	7000 3100 7000 3000
 Wire Wire Line
-	7100 3500 6500 3500
+	7100 3500 7000 3500
 Text Label 6550 3500 0    50   ~ 0
 ~reset~
@@
 led2_mosi
 Text Label 1600 5850 0    50   ~ 0
-led3_miso
+led4_miso
 Text Label 1600 6050 0    50   ~ 0
-led4_sck
+led3_sck
 Text Label 1600 6150 0    50   ~ 0
 ~reset~
@@
 led2_mosi
 Text Label 8800 2000 0    50   ~ 0
-led3_miso
+led3_sck
 Text Label 8800 2500 0    50   ~ 0
-led4_sck
+led4_miso
 Wire Wire Line
 	8750 1000 9350 1000
@@
 Wire Wire Line
 	7250 6000 7500 6000
+Connection ~ 7000 3500
+Wire Wire Line
+	7000 3500 7000 3400
+Wire Wire Line
+	7000 3500 6500 3500
 $EndSCHEMATC
