File: Devices/LedBar/Hardware/Boards/MainBoard/Microcontroller.sch (KiCad schematic (older format))
At the start: 29 parts, among them J401 AVR-ISP-6, SW401 reset, U401 ATmega48PV-10AU-arduino, Y401 14.7456Mhz

Commit message: Work in progress
Parts:
- added TP407, TP408: gnd, AmbientLight:TestPoint_Pad_D1.0mm, symbol Connector:TestPoint
Connections:
- wire segments 99 -> 101
Changed lines of the file:
@@
 Wire Wire Line
 	7000 3500 6500 3500
+$Comp
+L power:GND #PWR0104
+U 1 1 60E286D3
+P 5500 4100
+F 0 "#PWR0104" H 5500 3850 50  0001 C CNN
+F 1 "GND" H 5505 3927 50  0000 C CNN
+F 2 "" H 5500 4100 50  0001 C CNN
+F 3 "" H 5500 4100 50  0001 C CNN
+	1    5500 4100
+	1    0    0    -1
+$EndComp
+Wire Wire Line
+	5500 3950 5500 4100
+$Comp
+L Connector:TestPoint TP407
+U 1 1 60E27489
+P 5500 3950
+F 0 "TP407" H 5442 3976 50  0000 R CNN
+F 1 "gnd" H 5442 4067 50  0000 R CNN
+F 2 "AmbientLight:TestPoint_Pad_D1.0mm" H 5700 3950 50  0001 C CNN
+F 3 "~" H 5700 3950 50  0001 C CNN
+	1    5500 3950
+	1    0    0    -1
+$EndComp
+$Comp
+L power:GND #PWR0106
+U 1 1 60E6D7A2
+P 8150 5050
+F 0 "#PWR0106" H 8150 4800 50  0001 C CNN
+F 1 "GND" H 8155 4877 50  0000 C CNN
+F 2 "" H 8150 5050 50  0001 C CNN
+F 3 "" H 8150 5050 50  0001 C CNN
+	1    8150 5050
+	1    0    0    -1
+$EndComp
+Wire Wire Line
+	8150 4900 8150 5050
+$Comp
+L Connector:TestPoint TP408
+U 1 1 60E6D7A9
+P 8150 4900
+F 0 "TP408" H 8092 4926 50  0000 R CNN
+F 1 "gnd" H 8092 5017 50  0000 R CNN
+F 2 "AmbientLight:TestPoint_Pad_D1.0mm" H 8350 4900 50  0001 C CNN
+F 3 "~" H 8350 4900 50  0001 C CNN
+	1    8150 4900
+	1    0    0    -1
+$EndComp
 $EndSCHEMATC
