File: Devices/LedBar/Hardware/Boards/MainBoard/0-10V.sch (KiCad schematic (older format))
At the start: 24 parts, among them J601 0-10V(1), J602 0-10V(2), U601 LM393

Commit message: Renamed CenterBoard to MainBoard
Parts:
- R609: footprint (none) -> Resistor_SMD:R_0805_2012Metric_Pad1.20x1.40mm_HandSolder
Changed lines of the file:
@@
 encoding utf-8
 Sheet 6 6
-Title ""
-Date ""
-Rev ""
-Comp ""
+Title "LedBar - MainBoard"
+Date "2021-04-25"
+Rev "0.1"
+Comp "Roel Drost"
 Comment1 ""
 Comment2 ""
@@
 F 0 "R609" H 7930 2954 50  0000 R CNN
 F 1 "100" H 7930 3045 50  0000 R CNN
-F 2 "" V 7930 3000 50  0001 C CNN
+F 2 "Resistor_SMD:R_0805_2012Metric_Pad1.20x1.40mm_HandSolder" V 7930 3000 50  0001 C CNN
 F 3 "~" H 8000 3000 50  0001 C CNN
 	1    8000 3000

Commit message: Placing and routing
Parts:
- removed J602: 0-10V(2), AmbientLight:15EDGRC-3.5-2P, symbol Connector_Generic:Conn_01x02
- C606: value 10uF/16V -> 4.7uF/16V
- J601: footprint AmbientLight:15EDGRC-3.5-2P -> AmbientLight:15EDGRC-3.5-3P; symbol Connector_Generic:Conn_01x02 -> Connector_Generic:Conn_01x03
Connections:
- net GND: now also J601.3 (Pin_3); no longer J601.2 (Pin_2)
- net at C604.1, R606.2, R607.1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: now also J601.2 (Pin_2)
Other:
- moved on the sheet: C601, C602, C603, C604, C605, C606, R601, R602, R603, R604, R605, R606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

Commit message: Added Brown-out detection
Parts:
- removed C602: 1uF, Capacitor_SMD:C_0805_2012Metric_Pad1.18x1.45mm_HandSolder, symbol Device:C
- removed C604: 0.1uF, Capacitor_SMD:C_0805_2012Metric_Pad1.18x1.45mm_HandSolder, symbol Device:C
- removed R602: 100k, Resistor_SMD:R_0805_2012Metric_Pad1.20x1.40mm_HandSolder, symbol Device:R
- removed R606: 1k, Resistor_SMD:R_0805_2012Metric_Pad1.20x1.40mm_HandSolder, symbol Device:R
- removed R607, R608: 10k, Resistor_SMD:R_0805_2012Metric_Pad1.20x1.40mm_HandSolder, symbol Device:R
- removed TP602: pwm2, AmbientLight:TestPoint_Pad_D1.0mm, symbol Connector:TestPoint
- removed TP604: a2, AmbientLight:TestPoint_Pad_D1.0mm, symbol Connector:TestPoint
- removed TP606: ao2, AmbientLight:TestPoint_Pad_D1.0mm, symbol Connector:TestPoint
- added D501: 4V7, symbol Device:D_Zener
- added D502: Blue, symbol Device:LED
- added R501, R506, R507: 10k, Resistor_SMD:R_0805_2012Metric_Pad1.20x1.40mm_HandSolder, symbol Device:R
- added R502: 15k, Resistor_SMD:R_0805_2012Metric_Pad1.20x1.40mm_HandSolder, symbol Device:R
- added R503, R504: 18k, Resistor_SMD:R_0805_2012Metric_Pad1.20x1.40mm_HandSolder, symbol Device:R
- added R505: 150k, Resistor_SMD:R_0805_2012Metric_Pad1.20x1.40mm_HandSolder, symbol Device:R
- added TP502: BO, symbol Connector:TestPoint
- J601: footprint AmbientLight:15EDGRC-3.5-3P -> AmbientLight:15EDGRC-3.5-2P; symbol Connector_Generic:Conn_01x03 -> Connector_Generic:Conn_01x02
Connections:
- net +12V: now also R501.1, R503.1
- net GND: now also J601.2 (Pin_2), D501.2 (A), R502.2; no longer J601.3 (Pin_3)
- net at C601.1, R601.1, TP603.1: now also U601.5 (+); no longer U601.3 (+)
- net at C603.1, J601.1 (Pin_1), R603.2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: now also U601.7; no longer U601.1
- net at R604.2, R605.1: now also U601.6 (_); no longer U601.2 (-)
- new net: R501.2, R502.1, U601.2 (-)
- new net: R503.2, R504.1, R505.2, U601.3 (+)
- new net: D501.1 (K), R504.2
- new net: D502.2 (A), R507.2
- new net +5V: R506.1, R507.1
- new net ~Brown_out~: D502.1 (K), R505.1, R506.2, TP502.1, U601.1
Other:
- note added: "When the +12V line rise above 11.1V the BO (brown-out) line will change to Low.\nWhen the +12V line drops below 10.2V the BO line will change to high."
- moved on the sheet: U601A, U601B

Commit message: Moved brown-out to it own sheet
Parts:
- removed C605: 0.1uF, Capacitor_SMD:C_0805_2012Metric_Pad1.18x1.45mm_HandSolder, symbol Device:C
- removed C606: 4.7uF/16V, Capacitor_Tantalum_SMD:CP_EIA-6032-28_Kemet-C_Pad2.25x2.35mm_HandSolder, symbol Device:CP
- removed D501: 4V7, symbol Device:D_Zener
- removed D502: Blue, symbol Device:LED
- removed R501, R506, R507: 10k, Resistor_SMD:R_0805_2012Metric_Pad1.20x1.40mm_HandSolder, symbol Device:R
- removed R502: 15k, Resistor_SMD:R_0805_2012Metric_Pad1.20x1.40mm_HandSolder, symbol Device:R
- removed R503, R504: 18k, Resistor_SMD:R_0805_2012Metric_Pad1.20x1.40mm_HandSolder, symbol Device:R
- removed R505: 150k, Resistor_SMD:R_0805_2012Metric_Pad1.20x1.40mm_HandSolder, symbol Device:R
- removed R609: 100, Resistor_SMD:R_0805_2012Metric_Pad1.20x1.40mm_HandSolder, symbol Device:R
- removed TP502: BO, symbol Connector:TestPoint
- removed unit 1 of U601
- removed unit 3 of U601
- renumbered U601 to U701
Other:
- note removed: "When the +12V line rise above 11.1V the BO (brown-out) line will change to Low.\nWhen the +12V line drops below 10.2V the BO line will change to high."

Commit message: Added footprints for brown-out circuit
Other:
- moved on the sheet: C601, C603, J601, R601, R603, R604, R605, TP601, TP603, TP605, U701B

Commit message: Routed 0-10V and brownout circuits
Connections:
- net a1: now reaches C601.1, R601.1, TP603.1, U701.5 (+)
Changed lines of the file:
@@
 Wire Wire Line
 	6650 4000 7600 4000
+Text Label 4900 3900 0    50   ~ 0
+a1
 $EndSCHEMATC
