File: Devices/LedBar/Hardware/Boards/MainBoard/Brown-out.sch (KiCad schematic (older format))
At the start: 14 parts, among them U701 LM393

Commit message: Added footprints for brown-out circuit
Parts:
- D701: footprint (none) -> Diode_SMD:D_1206_3216Metric_Pad1.42x1.75mm_HandSolder
- D702: footprint (none) -> LED_SMD:LED_0805_2012Metric_Pad1.15x1.40mm_HandSolder
- R704: value 18k -> 10k
- TP701: footprint (none) -> AmbientLight:TestPoint_Pad_D1.0mm
Changed lines of the file:
@@
 AR Path="/608C0E66/6095EA74" Ref="R?"  Part="1"
 AR Path="/6094F41A/6095EA74" Ref="R705"  Part="1"
-F 0 "R705" V 5600 4350 50  0000 L CNN
+F 0 "R705" V 5600 4300 50  0000 L CNN
 F 1 "150k" V 5400 4400 50  0000 C CNN
 F 2 "Resistor_SMD:R_0805_2012Metric_Pad1.20x1.40mm_HandSolder" V 5430 4400 50  0001 C CNN
@@
 AR Path="/6094F41A/6095EA7A" Ref="R704"  Part="1"
 F 0 "R704" H 5070 4696 50  0000 L CNN
-F 1 "18k" H 5070 4605 50  0000 L CNN
+F 1 "10k" H 5070 4605 50  0000 L CNN
 F 2 "Resistor_SMD:R_0805_2012Metric_Pad1.20x1.40mm_HandSolder" V 4930 4650 50  0001 C CNN
 F 3 "~" H 5000 4650 50  0001 C CNN
@@
 F 0 "D701" V 4954 5230 50  0000 L CNN
 F 1 "4V7" V 5045 5230 50  0000 L CNN
-F 2 "" H 5000 5150 50  0001 C CNN
+F 2 "Diode_SMD:D_1206_3216Metric_Pad1.42x1.75mm_HandSolder" H 5000 5150 50  0001 C CNN
 F 3 "~" H 5000 5150 50  0001 C CNN
 	1    5000 5150
@@
 F 0 "D702" V 6539 3782 50  0000 R CNN
 F 1 "Blue" V 6448 3782 50  0000 R CNN
-F 2 "" H 6500 3900 50  0001 C CNN
+F 2 "LED_SMD:LED_0805_2012Metric_Pad1.15x1.40mm_HandSolder" H 6500 3900 50  0001 C CNN
 F 3 "~" H 6500 3900 50  0001 C CNN
 	1    6500 3900
@@
 F 0 "TP701" H 5942 4526 50  0000 R CNN
 F 1 "BO" H 5942 4617 50  0000 R CNN
-F 2 "" H 6200 4500 50  0001 C CNN
+F 2 "AmbientLight:TestPoint_Pad_D1.0mm" H 6200 4500 50  0001 C CNN
 F 3 "~" H 6200 4500 50  0001 C CNN
 	1    6000 4500

Commit message: Work in progress
Connections:
- net +12V: no longer R701.1, R703.1
- net +12VA: now also R701.1, R703.1
Changed lines of the file:
@@
 Wire Wire Line
 	6500 4400 6850 4400
-Wire Wire Line
-	4750 2650 4750 2900
 Connection ~ 4750 2900
 Wire Wire Line
@@
 Wire Wire Line
 	6000 4500 6000 4400
-$Comp
-L power:+12V #PWR?
-U 1 1 6095EAD6
-P 4750 2650
-AR Path="/608C0E66/6095EAD6" Ref="#PWR?"  Part="1"
-AR Path="/6094F41A/6095EAD6" Ref="#PWR0702"  Part="1"
-F 0 "#PWR0702" H 4750 2500 50  0001 C CNN
-F 1 "+12V" H 4765 2823 50  0000 C CNN
-F 2 "" H 4750 2650 50  0001 C CNN
-F 3 "" H 4750 2650 50  0001 C CNN
-	1    4750 2650
-	1    0    0    -1
-$EndComp
 Connection ~ 6500 4400
 $Comp
@@
 	0    1    1    0
 $EndComp
+$Comp
+L power:+12VA #PWR?
+U 1 1 60E43840
+P 4750 2650
+AR Path="/608C0E66/60E43840" Ref="#PWR?"  Part="1"
+AR Path="/6094F41A/60E43840" Ref="#PWR0105"  Part="1"
+F 0 "#PWR0105" H 4750 2500 50  0001 C CNN
+F 1 "+12VA" H 4765 2823 50  0000 C CNN
+F 2 "" H 4750 2650 50  0001 C CNN
+F 3 "" H 4750 2650 50  0001 C CNN
+	1    4750 2650
+	1    0    0    -1
+$EndComp
+Wire Wire Line
+	4750 2650 4750 2900
 $EndSCHEMATC
