File: Devices/LedBar/Hardware/Boards/MainBoard/Pca.sch (KiCad schematic (older format))
At the start: 26 parts, among them J501 Left, J502 Center, J503 Right, Q501 Si2302DS, Q502 Si2302DS, Q503 Si2302DS, Q504 Si2302DS, Q505 Si2302DS, Q506 Si2302DS, Q507 Si2302DS, Q508 Si2302DS, Q509 Si2302DS, Q510 Si2302DS, Q511 Si2302DS, Q512 Si2302DS, Q513 Si2302DS, Q514 Si2302DS, Q515 Si2302DS, Q516 Si2302DS, U501 PCA9685PW

Commit message: Added RGBW-wire-solder-pads, removed ground-tie, routing...
Parts:
- J501: footprint Connector_PinHeader_2.00mm:PinHeader_1x05_P2.00mm_Vertical -> AmbientLight:RGBW-wire-solder-pads-L
- J503: footprint Connector_PinHeader_2.00mm:PinHeader_1x05_P2.00mm_Vertical -> AmbientLight:RGBW-wire-solder-pads-R
Changed lines of the file:
@@
 F 0 "J501" H 2418 5767 50  0000 C CNN
 F 1 "Left" H 2418 5676 50  0000 C CNN
-F 2 "Connector_PinHeader_2.00mm:PinHeader_1x05_P2.00mm_Vertical" H 2500 5350 50  0001 C CNN
+F 2 "AmbientLight:RGBW-wire-solder-pads-L" H 2500 5350 50  0001 C CNN
 F 3 "~" H 2500 5350 50  0001 C CNN
 	1    2500 5350
@@
 Wire Wire Line
 	4000 5900 3750 5900
-$Comp
-L power:GNDPWR #PWR0505
-U 1 1 608E9633
-P 4000 6100
-F 0 "#PWR0505" H 4000 5900 50  0001 C CNN
-F 1 "GNDPWR" H 4004 5946 50  0000 C CNN
-F 2 "" H 4000 6050 50  0001 C CNN
-F 3 "" H 4000 6050 50  0001 C CNN
-	1    4000 6100
-	1    0    0    -1
-$EndComp
 $Comp
 L Connector_Generic:Conn_02x07_Odd_Even J502
@@
 F 0 "J503" H 9580 5392 50  0000 L CNN
 F 1 "Right" H 9580 5301 50  0000 L CNN
-F 2 "Connector_PinHeader_2.00mm:PinHeader_1x05_P2.00mm_Vertical" H 9500 5350 50  0001 C CNN
+F 2 "AmbientLight:RGBW-wire-solder-pads-R" H 9500 5350 50  0001 C CNN
 F 3 "~" H 9500 5350 50  0001 C CNN
 	1    9500 5350
@@
 Wire Wire Line
 	7500 5050 7500 5150
+$Comp
+L power:GNDPWR #PWR0505
+U 1 1 608E9633
+P 4000 6100
+F 0 "#PWR0505" H 4000 5900 50  0001 C CNN
+F 1 "GNDPWR" H 4004 5946 50  0000 C CNN
+F 2 "" H 4000 6050 50  0001 C CNN
+F 3 "" H 4000 6050 50  0001 C CNN
+	1    4000 6100
+	1    0    0    -1
+$EndComp
 $EndSCHEMATC

Commit message: Work in progress
Parts:
- added TP502: strip1_w, AmbientLight:TestPoint_Pad_D1.0mm, symbol Connector:TestPoint
- added TP503: strip1_w_out, AmbientLight:TestPoint_Pad_D1.0mm, symbol Connector:TestPoint
- added TP504: gnd, AmbientLight:TestPoint_Pad_D1.0mm, symbol Connector:TestPoint
Connections:
- wire segments 138 -> 139
Changed lines of the file:
@@
 $EndComp
 Wire Wire Line
-	10000 1200 10000 1350
+	10000 1200 10000 1300
 Wire Wire Line
 	10000 800  10500 800
@@
 	1    0    0    -1
 $EndComp
+$Comp
+L Connector:TestPoint TP?
+U 1 1 60E72D62
+P 9250 1000
+AR Path="/608B1159/60E72D62" Ref="TP?"  Part="1"
+AR Path="/608B2A01/60E72D62" Ref="TP502"  Part="1"
+F 0 "TP502" V 9150 1200 50  0000 R CNN
+F 1 "strip1_w" V 9350 1300 50  0000 R CNN
+F 2 "AmbientLight:TestPoint_Pad_D1.0mm" H 9450 1000 50  0001 C CNN
+F 3 "~" H 9450 1000 50  0001 C CNN
+	1    9250 1000
+	0    -1   -1   0
+$EndComp
+$Comp
+L Connector:TestPoint TP?
+U 1 1 60E8F95C
+P 10500 800
+AR Path="/608B1159/60E8F95C" Ref="TP?"  Part="1"
+AR Path="/608B2A01/60E8F95C" Ref="TP503"  Part="1"
+F 0 "TP503" V 10400 1000 50  0000 R CNN
+F 1 "strip1_w_out" V 10500 1450 50  0000 R CNN
+F 2 "AmbientLight:TestPoint_Pad_D1.0mm" H 10700 800 50  0001 C CNN
+F 3 "~" H 10700 800 50  0001 C CNN
+	1    10500 800
+	0    1    1    0
+$EndComp
+$Comp
+L Connector:TestPoint TP?
+U 1 1 60EE1BB4
+P 10000 1300
+AR Path="/608B1159/60EE1BB4" Ref="TP?"  Part="1"
+AR Path="/608B2A01/60EE1BB4" Ref="TP504"  Part="1"
+F 0 "TP504" V 9900 1650 50  0000 R CNN
+F 1 "gnd" V 10000 1600 50  0000 R CNN
+F 2 "AmbientLight:TestPoint_Pad_D1.0mm" H 10200 1300 50  0001 C CNN
+F 3 "~" H 10200 1300 50  0001 C CNN
+	1    10000 1300
+	0    1    1    0
+$EndComp
+Connection ~ 10000 1300
+Wire Wire Line
+	10000 1300 10000 1350
 $EndSCHEMATC
